Commit message: add scripts directory to share remove joint_state and joint_state_gui from rviz launch moves gazebo launches back to active directory adds main entry point with swerve.launch.py fixes zero inertia at wheel module links in swerve URDF tweaks rviz config to add markers tweaks plane URDF to add small mass

File: swerve_drive/urdf/plane.urdf (robot description, URDF)
Before this commit: robot plane, 1 links, 0 joints
Links:
- link planeLink: mass .0 -> 1

File: swerve_drive/urdf/swerve.urdf (robot description, URDF)
Before this commit: robot swerve, 8 links, 7 joints
Links:
- link mod_1: mass 0.00001 -> 0.4545
- link mod_2: mass 0.00001 -> 0.4545
- link mod_3: mass 0.00001 -> 0.4545
- link wheel_1: mass 0.11364 -> 0.4545
- link wheel_2: mass 0.11364 -> 0.4545
- link wheel_3: mass 0.11364 -> 0.4545
Joints:
- removed joint base_footprint_link
- added joint base_footprint_joint: type fixed, parent base_link, child base_footprint, origin xyz=0 0 ${-wheel_offset - r_wheel} rpy=0 0 0, axis 0 0 1
