Commit message: preliminary joint PID plugin, needs debug

File: swerve_drive/urdf/swerve_macros.xacro (robot description, xacro)
@@ -63,12 +63,28 @@
     <xacro:macro name="v5_motor_macro" params="joint_name link_name gear_ratio">
         <plugin name="${link_name}_motor_plugin" filename="libgazebo_motor_plugin.so">
-        <joint_name>${joint_name}</joint_name>
-        <link_name>${link_name}</link_name>
-        <free_speed>130</free_speed>
-        <stall_torque>4.5</stall_torque>
-        <free_current>0.1</free_current>
-        <stall_current>4.5</stall_current>
-        <nominal_voltage>12.8</nominal_voltage>
-        <gear_ratio>${gear_ratio}</gear_ratio>
+            <joint_name>${joint_name}</joint_name>
+            <link_name>${link_name}</link_name>
+            <free_speed>130</free_speed>
+            <stall_torque>4.5</stall_torque>
+            <free_current>0.1</free_current>
+            <stall_current>4.5</stall_current>
+            <nominal_voltage>12.8</nominal_voltage>
+            <gear_ratio>${gear_ratio}</gear_ratio>
+        </plugin>
+    </xacro:macro>
+    <!-- Motor PID Macro -->
+    <xacro:macro name="joint_pid_macro" params="joint_name link_name gear_ratio position_gain vel_gain accel_gain">
+        <plugin name="${link_name}_joint_pid_plugin" filename="libgazebo_joint_pid_plugin.so">
+            <joint_name>${joint_name}</joint_name>
+            <link_name>${link_name}</link_name>
+            <position_gain>${position_gain}</position_gain>
+            <vel_gain>${vel_gain}</vel_gain>
+            <accel_gain>${accel_gain}</accel_gain>
+            <free_speed>130</free_speed>
+            <stall_torque>4.5</stall_torque>
+            <free_current>0.1</free_current>
+            <stall_current>4.5</stall_current>
+            <nominal_voltage>12.8</nominal_voltage>
+            <gear_ratio>${gear_ratio}</gear_ratio>
         </plugin>
     </xacro:macro>
