Commit message: add plane urdf fix missing inertia in swerve urdf

File: swerve_drive/urdf/swerve.urdf (robot description, URDF)
Before this commit: robot swerve, 8 links, 7 joints
Links:
- link base_footprint: mass None -> 0.00001

Commit message: fixes wheel friction issues by decreasing collision width to point starts integrating direction into wheel motor model adds publishers for torque and speed to swerve gz plugin

File: swerve_drive/urdf/swerve.urdf (robot description, URDF)
Before this commit: robot swerve, 8 links, 7 joints
Links:
- link wheel_1: geometry collision cylinder length=${width_wheel/8} radius=${r_wheel}; visual cylinder length=${width_wheel} radius=${r_wheel}
- link wheel_2: geometry collision cylinder length=${width_wheel/8} radius=${r_wheel}; visual cylinder length=${width_wheel} radius=${r_wheel}
- link wheel_3: geometry collision cylinder length=${width_wheel/8} radius=${r_wheel}; visual cylinder length=${width_wheel} radius=${r_wheel}

Commit message: tweak swerve urdf makes field walls static changes swerve gz plugin output topics to true speed

File: swerve_drive/urdf/swerve.urdf (robot description, URDF)
Before this commit: robot swerve, 8 links, 7 joints
Links:
- link base_link: mass 7 -> 10
- link wheel_1: geometry collision cylinder length=${width_wheel/4} radius=${r_wheel}; visual cylinder length=${width_wheel} radius=${r_wheel}
- link wheel_2: geometry collision cylinder length=${width_wheel/4} radius=${r_wheel}; visual cylinder length=${width_wheel} radius=${r_wheel}
- link wheel_3: geometry collision cylinder length=${width_wheel/4} radius=${r_wheel}; visual cylinder length=${width_wheel} radius=${r_wheel}
Joints:
- joint base_footprint_joint: origin xyz=0 0 ${-wheel_offset - r_wheel} rpy=0 0 0 -> xyz=0 0 ${- r_wheel} rpy=0 0 0
- joint driveshaft_1: origin xyz=0 0 -${wheel_offset} rpy=${90*d2r} 0 ${90*d2r} -> xyz=0 0 0 rpy=${90*d2r} 0 ${90*d2r}
- joint driveshaft_2: origin xyz=0 0 -${wheel_offset} rpy=${90*d2r} 0 ${90*d2r} -> xyz=0 0 0 rpy=${90*d2r} 0 ${90*d2r}
- joint driveshaft_3: origin xyz=0 0 -${wheel_offset} rpy=${90*d2r} 0 ${90*d2r} -> xyz=0 0 0 rpy=${90*d2r} 0 ${90*d2r}

Commit message: refactors swerve plugin to be single motor refactors motor plugin to be fully configurable from URDF Fixes torque and current calculations for dc motor model Adds physics config to world model Adds torsional friction to wheel steering Splits swerve URDF into macros

File: swerve_drive/urdf/swerve.urdf (robot description, URDF)
Before this commit: robot swerve, 8 links, 7 joints
Links:
- removed link mod_1
- removed link mod_2
- removed link mod_3
- removed link wheel_1
- removed link wheel_2
- removed link wheel_3
Joints:
- removed joint pivot_1
- removed joint pivot_2
- removed joint pivot_3
- added joint steering_1: type continuous, parent base_link, child mod_1, origin xyz=${l_wheel*0.866} ${l_wheel/2} 0 rpy=0 0 0, axis 0 0 1
- added joint steering_2: type continuous, parent base_link, child mod_2, origin xyz=${-l_wheel*0.866} ${l_wheel/2} 0 rpy=0 0 0, axis 0 0 1
- added joint steering_3: type continuous, parent base_link, child mod_3, origin xyz=0 ${-l_wheel} 0 rpy=0 0 0, axis 0 0 1

Commit message: adds LIDAR to simulator and RVIZ small refactor in start_sim scripts adds simulator back to swerve launch adds launch script for easy entry point

File: swerve_drive/urdf/swerve.urdf (robot description, URDF)
Before this commit: robot swerve, 2 links, 7 joints
Links:
- added link lidar_link, mass 0.125; visual cylinder length=0.025 radius=0.0508
Joints:
- added joint lidar_joint: type fixed, parent base_link, child lidar_link, origin xyz=0 0 0.1 rpy=0 0 0
