Commit message: migrates simulation nodes to ghost_sim package reorganizes URDF configuration moves all simulation specific URDF to ghost_sim consolidates launch files using CLI args with ROS Launch splits build script for hardware specific build (no sim)

File: ghost_ros/urdf/ghost1.xacro (robot description, xacro)
@@ -1,4 +1,4 @@
 <?xml version="1.0"?>
-<robot name="swerve" xmlns:xacro="http://ros.org/wiki/xacro">
+<robot name="ghost1" xmlns:xacro="http://ros.org/wiki/xacro">
     <xacro:include filename="$(find ghost_ros)/urdf/swerve_macros.xacro"/>
     <xacro:property name="l_wheel" value="0.2286"/> <!-- 9" center to wheel modules-->
@@ -108,57 +108,3 @@
         <origin xyz="0 0 0.1" rpy="0 0 0"/>
     </joint>
-    <gazebo reference="lidar_link">
-        <sensor name="lidar" type="ray">
-            <always_on>true</always_on>
-            <visualize>true</visualize>
-            <update_rate>5</update_rate>
-            <ray>
-            <scan>
-                <horizontal>
-                <samples>360</samples>
-                <resolution>1.000000</resolution>
-                <min_angle>0.000000</min_angle>
-                <max_angle>6.280000</max_angle>
-                </horizontal>
-            </scan>
-            <range>
-                <min>0.120000</min>
-                <max>3.5</max>
-                <resolution>0.015000</resolution>
-            </range>
-            <noise>
-                <type>gaussian</type>
-                <mean>0.0</mean>
-                <stddev>0.01</stddev>
-            </noise>
-            </ray>
-            <plugin name="scan" filename="libgazebo_ros_ray_sensor.so">
-            <ros>
-                <remapping>~/out:=scan</remapping>
-            </ros>
-            <output_type>sensor_msgs/LaserScan</output_type>
-            <frame_name>lidar_link</frame_name>
-            </plugin>
-        </sensor>
-    </gazebo>
-    <!-- Gazebo Plugins -->
-    <gazebo>
-        <!-- Joint State Publisher -->
-        <plugin name="gazebo_ros_joint_state_publisher" filename="libgazebo_ros_joint_state_publisher.so">
-            <update_rate>100</update_rate>
-            <joint_name>steering_1</joint_name>
-            <joint_name>steering_2</joint_name>
-            <joint_name>steering_3</joint_name>
-            <joint_name>driveshaft_1</joint_name>
-            <joint_name>driveshaft_2</joint_name>
-            <joint_name>driveshaft_3</joint_name>
-        </plugin>
-        <!-- Motor Models -->
-        <xacro:v5_motor_macro joint_name="steering_1" link_name="mod_1" gear_ratio="1.0"></xacro:v5_motor_macro>
-        <xacro:v5_motor_macro joint_name="steering_2" link_name="mod_2" gear_ratio="1.0"></xacro:v5_motor_macro>
-        <xacro:v5_motor_macro joint_name="steering_3" link_name="mod_3" gear_ratio="1.0"></xacro:v5_motor_macro>
-        <xacro:v5_motor_macro joint_name="driveshaft_1" link_name="wheel_1" gear_ratio="6.0"></xacro:v5_motor_macro>
-        <xacro:v5_motor_macro joint_name="driveshaft_2" link_name="wheel_2" gear_ratio="6.0"></xacro:v5_motor_macro>
-        <xacro:v5_motor_macro joint_name="driveshaft_3" link_name="wheel_3" gear_ratio="6.0"></xacro:v5_motor_macro>
-    </gazebo>
 </robot>

File: ghost_ros/urdf/swerve_macros.xacro (robot description, xacro)
@@ -60,32 +60,3 @@
     </gazebo>
     </xacro:macro>
-    <!-- Motor Macro -->
-    <xacro:macro name="v5_motor_macro" params="joint_name link_name gear_ratio">
-        <plugin name="${link_name}_motor_plugin" filename="libgazebo_motor_plugin.so">
-            <joint_name>${joint_name}</joint_name>
-            <link_name>${link_name}</link_name>
-            <free_speed>130</free_speed>
-            <stall_torque>4.5</stall_torque>
-            <free_current>0.1</free_current>
-            <stall_current>4.5</stall_current>
-            <nominal_voltage>12.8</nominal_voltage>
-            <gear_ratio>${gear_ratio}</gear_ratio>
-        </plugin>
-    </xacro:macro>
-    <!-- Motor PID Macro -->
-    <xacro:macro name="joint_pid_macro" params="joint_name link_name gear_ratio position_gain vel_gain accel_gain">
-        <plugin name="${link_name}_joint_pid_plugin" filename="libgazebo_joint_pid_plugin.so">
-            <joint_name>${joint_name}</joint_name>
-            <link_name>${link_name}</link_name>
-            <position_gain>${position_gain}</position_gain>
-            <vel_gain>${vel_gain}</vel_gain>
-            <accel_gain>${accel_gain}</accel_gain>
-            <free_speed>130</free_speed>
-            <stall_torque>4.5</stall_torque>
-            <free_current>0.1</free_current>
-            <stall_current>4.5</stall_current>
-            <nominal_voltage>12.8</nominal_voltage>
-            <gear_ratio>${gear_ratio}</gear_ratio>
-        </plugin>
-    </xacro:macro>
 </robot>

Commit message: adds URDFs including realsense link

File: ghost_ros/urdf/ghost1.xacro (robot description, xacro)
@@ -3,5 +3,5 @@
     <xacro:include filename="$(find ghost_ros)/urdf/swerve_macros.xacro"/>
     <xacro:property name="l_wheel" value="0.2286"/> <!-- 9" center to wheel modules-->
-    <xacro:property name="r_wheel" value="0.034925"/> <!-- 2.75" wheel diameter-->
+    <xacro:property name="r_wheel" value="0.034925"/> <!-- 1.375" wheel radius-->
     <xacro:property name="width_wheel" value="0.0254"/> <!-- 1" wheel width-->
     <xacro:property name="com_radius" value="0.02"/>
@@ -92,5 +92,5 @@
     <link name="lidar_link">
         <inertial>
-            <origin xyz="0.2 0 0.24" rpy="0 0 0"/>
+            <origin xyz="0.0 0 0.0" rpy="0 0 0"/>
             <mass value="0.125"/>
             <inertia ixx="0.001"  ixy="0"  ixz="0" iyy="0.001" iyz="0" izz="0.001" />
@@ -108,3 +108,15 @@
         <origin xyz="0 0 0.1" rpy="0 0 0"/>
     </joint>
+    <link name="camera_link">
+        <inertial>
+            <origin xyz="0.0 0 0.0" rpy="0 0 0"/>
+            <mass value="0.125"/>
+            <inertia ixx="0.001"  ixy="0"  ixz="0" iyy="0.001" iyz="0" izz="0.001" />
+        </inertial>
+    </link>
+    <joint name="camera_joint" type="fixed">
+        <parent link="base_link"/>
+        <child link="camera_link"/>
+        <origin xyz="${l_wheel/2} 0 0.33" rpy="0 0 0"/>
+    </joint>
 </robot>

File: ghost_sim/urdf/ghost1_sim_pid.xacro (robot description, xacro)
@@ -5,5 +5,10 @@
     <!-- Import Primary Robot URDF -->
     <xacro:include filename="$(find ghost_ros)/urdf/ghost1.xacro"/>
+    <!-- Add Sensors -->
     <xacro:lidar_macro link_name="lidar_link" topic_name="scan"></xacro:lidar_macro>
+    <xacro:include filename="$(find realsense2_description)/urdf/_d435i.urdf.xacro"/>
+    <xacro:sensor_d435i parent="camera_link" >
+        <origin xyz="0 0 0" rpy="0 -0.7853975 0"/>
+    </xacro:sensor_d435i>
     <!-- Gazebo Plugins -->
     <gazebo>

File: ghost_sim/urdf/ghost1_sim_voltage.xacro (robot description, xacro)
@@ -5,5 +5,10 @@
     <!-- Import Primary Robot URDF -->
     <xacro:include filename="$(find ghost_ros)/urdf/ghost1.xacro"/>
+    <!-- Add Sensors -->
     <xacro:lidar_macro link_name="lidar_link" topic_name="scan"></xacro:lidar_macro>
+    <xacro:include filename="$(find realsense2_description)/urdf/_d435i.urdf.xacro"/>
+    <xacro:sensor_d435i parent="camera_link" >
+        <origin xyz="0 0 0" rpy="0 -0.7853975 0"/>
+    </xacro:sensor_d435i>
     <!-- Gazebo Plugins -->
     <gazebo>

Commit message: adds imu macro adds camera link removes repeated urdf config in ghost_sim

File: ghost_ros/urdf/ghost1.xacro (robot description, xacro)
@@ -108,15 +108,27 @@
         <origin xyz="0 0 0.1" rpy="0 0 0"/>
     </joint>
-    <link name="camera_link">
+    <link name="camera_base_link">
         <inertial>
             <origin xyz="0.0 0 0.0" rpy="0 0 0"/>
             <mass value="0.125"/>
-            <inertia ixx="0.001"  ixy="0"  ixz="0" iyy="0.001" iyz="0" izz="0.001" />
+            <inertia ixx="0.001"  ixy="0.001"  ixz="0.001" iyy="0.001" iyz="0.001" izz="0.001" />
         </inertial>
     </link>
-    <joint name="camera_joint" type="fixed">
+    <joint name="camera_base_joint" type="fixed">
         <parent link="base_link"/>
-        <child link="camera_link"/>
-        <origin xyz="${l_wheel/2} 0 0.33" rpy="0 0 0"/>
+        <child link="camera_base_link"/>
+        <origin xyz="0 ${l_wheel/2} 0.33" rpy="0 0 1.570795"/>
+    </joint>
+    <link name="camera_view_link">
+        <inertial>
+            <origin xyz="0.0 0 0.0" rpy="0 0 0"/>
+            <mass value="0.125"/>
+            <inertia ixx="0.001"  ixy="0.001"  ixz="0.001" iyy="0.001" iyz="0.001" izz="0.001" />
+        </inertial>
+    </link>
+    <joint name="camera_view_joint" type="fixed">
+        <parent link="camera_base_link"/>
+        <child link="camera_view_link"/>
+        <origin xyz="0 0 0" rpy="0 0.7853975 0"/>
     </joint>
 </robot>

File: ghost_sim/urdf/ghost1_sim_pid.xacro (robot description, xacro)
@@ -1,26 +1,8 @@
 <?xml version="1.0"?>
 <robot name="ghost1" xmlns:xacro="http://ros.org/wiki/xacro">
-    <xacro:include filename="$(find ghost_sim)/urdf/macros/actuator_macros.xacro"/>
-    <xacro:include filename="$(find ghost_sim)/urdf/macros/sensor_macros.xacro"/>
     <!-- Import Primary Robot URDF -->
-    <xacro:include filename="$(find ghost_ros)/urdf/ghost1.xacro"/>
-    <!-- Add Sensors -->
-    <xacro:lidar_macro link_name="lidar_link" topic_name="scan"></xacro:lidar_macro>
-    <xacro:include filename="$(find realsense2_description)/urdf/_d435i.urdf.xacro"/>
-    <xacro:sensor_d435i parent="camera_link" >
-        <origin xyz="0 0 0" rpy="0 -0.7853975 0"/>
-    </xacro:sensor_d435i>
+    <xacro:include filename="$(find ghost_sim)/urdf/ghost1_sim_base.xacro"/>
     <!-- Gazebo Plugins -->
     <gazebo>
-        <!-- Joint State Publisher -->
-        <plugin name="gazebo_ros_joint_state_publisher" filename="libgazebo_ros_joint_state_publisher.so">
-            <update_rate>100</update_rate>
-            <joint_name>steering_1</joint_name>
-            <joint_name>steering_2</joint_name>
-            <joint_name>steering_3</joint_name>
-            <joint_name>driveshaft_1</joint_name>
-            <joint_name>driveshaft_2</joint_name>
-            <joint_name>driveshaft_3</joint_name>
-        </plugin>
         <!-- Motor Models -->
         <!-- 0.05 Steering -->

File: ghost_sim/urdf/ghost1_sim_voltage.xacro (robot description, xacro)
@@ -1,26 +1,8 @@
 <?xml version="1.0"?>
 <robot name="ghost1" xmlns:xacro="http://ros.org/wiki/xacro">
-    <xacro:include filename="$(find ghost_sim)/urdf/macros/actuator_macros.xacro"/>
-    <xacro:include filename="$(find ghost_sim)/urdf/macros/sensor_macros.xacro"/>
     <!-- Import Primary Robot URDF -->
-    <xacro:include filename="$(find ghost_ros)/urdf/ghost1.xacro"/>
-    <!-- Add Sensors -->
-    <xacro:lidar_macro link_name="lidar_link" topic_name="scan"></xacro:lidar_macro>
-    <xacro:include filename="$(find realsense2_description)/urdf/_d435i.urdf.xacro"/>
-    <xacro:sensor_d435i parent="camera_link" >
-        <origin xyz="0 0 0" rpy="0 -0.7853975 0"/>
-    </xacro:sensor_d435i>
+    <xacro:include filename="$(find ghost_sim)/urdf/ghost1_sim_base.xacro"/>
     <!-- Gazebo Plugins -->
     <gazebo>
-        <!-- Joint State Publisher -->
-        <plugin name="gazebo_ros_joint_state_publisher" filename="libgazebo_ros_joint_state_publisher.so">
-            <update_rate>100</update_rate>
-            <joint_name>steering_1</joint_name>
-            <joint_name>steering_2</joint_name>
-            <joint_name>steering_3</joint_name>
-            <joint_name>driveshaft_1</joint_name>
-            <joint_name>driveshaft_2</joint_name>
-            <joint_name>driveshaft_3</joint_name>
-        </plugin>
         <!-- Motor Models -->
         <xacro:v5_motor_macro joint_name="steering_1" link_name="mod_1" gear_ratio="1.0"></xacro:v5_motor_macro>

File: ghost_sim/urdf/macros/sensor_macros.xacro (robot description, xacro)
@@ -37,3 +37,73 @@
         </gazebo>
     </xacro:macro>
+    <xacro:macro name="imu_macro" params="parent_link">
+        <gazebo reference="${parent_link}">
+            <sensor name="imu_sensor" type="imu">
+            <plugin filename="libgazebo_ros_imu_sensor.so" name="imu_plugin">
+                <ros>
+                <namespace>/demo</namespace>
+                <remapping>~/out:=imu</remapping>
+                </ros>
+                <initial_orientation_as_reference>false</initial_orientation_as_reference>
+            </plugin>
+            <always_on>true</always_on>
+            <update_rate>100</update_rate>
+            <visualize>true</visualize>
+            <imu>
+                <angular_velocity>
+                <x>
+                    <noise type="gaussian">
+                    <mean>0.0</mean>
+                    <stddev>2e-4</stddev>
+                    <bias_mean>0.0000075</bias_mean>
+                    <bias_stddev>0.0000008</bias_stddev>
+                    </noise>
+                </x>
+                <y>
+                    <noise type="gaussian">
+                    <mean>0.0</mean>
+                    <stddev>2e-4</stddev>
+                    <bias_mean>0.0000075</bias_mean>
+                    <bias_stddev>0.0000008</bias_stddev>
+                    </noise>
+                </y>
+                <z>
+                    <noise type="gaussian">
+                    <mean>0.0</mean>
+                    <stddev>2e-4</stddev>
+                    <bias_mean>0.0000075</bias_mean>
+                    <bias_stddev>0.0000008</bias_stddev>
+                    </noise>
+                </z>
+                </angular_velocity>
+                <linear_acceleration>
+                <x>
+                    <noise type="gaussian">
+                    <mean>0.0</mean>
+                    <stddev>1.7e-2</stddev>
+                    <bias_mean>0.1</bias_mean>
+                    <bias_stddev>0.001</bias_stddev>
+                    </noise>
+                </x>
+                <y>
+                    <noise type="gaussian">
+                    <mean>0.0</mean>
+                    <stddev>1.7e-2</stddev>
+                    <bias_mean>0.1</bias_mean>
+                    <bias_stddev>0.001</bias_stddev>
+                    </noise>
+                </y>
+                <z>
+                    <noise type="gaussian">
+                    <mean>0.0</mean>
+                    <stddev>1.7e-2</stddev>
+                    <bias_mean>0.1</bias_mean>
+                    <bias_stddev>0.001</bias_stddev>
+                    </noise>
+                </z>
+                </linear_acceleration>
+            </imu>
+            </sensor>
+        </gazebo>
+    </xacro:macro>
 </robot>

Commit message: adds particle cloud visualization to RVIZ adds set_initial_pose in particle filter with RVIZ adds map loading to RVIZ fixes URDF to use proper base_link convention (Front-Left-Up)

File: ghost_ros/urdf/ghost1.xacro (robot description, xacro)
@@ -56,5 +56,5 @@
         <parent link="base_link"/>
         <child link="mod_1"/>
-        <origin xyz="${l_wheel*0.866} ${l_wheel/2} 0" rpy="0 0 0"/>
+        <origin xyz="${l_wheel/2} ${-l_wheel*0.866} 0" rpy="0 0 0"/>
         <axis xyz="0 0 1"/>
     </joint>
@@ -62,5 +62,5 @@
         <parent link="base_link"/>
         <child link="mod_2"/>
-        <origin xyz="${-l_wheel*0.866} ${l_wheel/2} 0" rpy="0 0 0"/>
+        <origin xyz="${l_wheel/2} ${l_wheel*0.866} 0" rpy="0 0 0"/>
         <axis xyz="0 0 1"/>
     </joint>
@@ -68,5 +68,5 @@
         <parent link="base_link"/>
         <child link="mod_3"/>
-        <origin xyz="0 ${-l_wheel} 0" rpy="0 0 0"/>
+        <origin xyz="${-l_wheel} 0 0" rpy="0 0 0"/>
         <axis xyz="0 0 1"/>
     </joint>
@@ -74,5 +74,5 @@
         <parent link="mod_1"/>
         <child link="wheel_1"/>
-        <origin xyz="0 0 0" rpy="${90*d2r} 0 ${90*d2r}"/>
+        <origin xyz="0 0 0" rpy="${90*d2r} 0 0"/>
         <axis xyz="0 0 1"/>
     </joint>
@@ -80,5 +80,5 @@
         <parent link="mod_2"/>
         <child link="wheel_2"/>
-        <origin xyz="0 0 0" rpy="${90*d2r} 0 ${90*d2r}"/>
+        <origin xyz="0 0 0" rpy="${90*d2r} 0 0"/>
         <axis xyz="0 0 1"/>
     </joint>
@@ -86,5 +86,5 @@
         <parent link="mod_3"/>
         <child link="wheel_3"/>
-        <origin xyz="0 0 0" rpy="${90*d2r} 0 ${90*d2r}"/>
+        <origin xyz="0 0 0" rpy="${90*d2r} 0 0"/>
         <axis xyz="0 0 1"/>
     </joint>
@@ -118,5 +118,5 @@
         <parent link="base_link"/>
         <child link="camera_base_link"/>
-        <origin xyz="0 ${l_wheel/2} 0.33" rpy="0 0 1.570795"/>
+        <origin xyz="${l_wheel/2} 0 0.33" rpy="0 0 0"/>
     </joint>
     <link name="camera_view_link">
