Commit message: refactors robot URDF to use left/right/back identifies removes Pose2D and adds preliminary GhostRobotState changes encoder angles to floats reverses encoders and changes update rate to 5ms refactors particle_filter_node to ghost_estimator_node refactors ghost_estimator config to have namespaces for particle filter and odometry fixes rear module port change from ESD board removal adds joint state publisher to ghost_estimator confirms working steering joint states

File: ghost_description/urdf/ghost1.xacro (robot description, xacro)
@@ -45,45 +45,45 @@
     </joint>
     <!-- Steering Modules -->
-    <xacro:steering_macro id="1"></xacro:steering_macro>
-    <xacro:steering_macro id="2"></xacro:steering_macro>
-    <xacro:steering_macro id="3"></xacro:steering_macro>
+    <xacro:steering_macro id="left"></xacro:steering_macro>
+    <xacro:steering_macro id="right"></xacro:steering_macro>
+    <xacro:steering_macro id="back"></xacro:steering_macro>
     <!-- Wheel Modules -->
-    <xacro:wheel_macro id="1" r_wheel="${r_wheel}" width_wheel="${width_wheel}" collision_factor="8"></xacro:wheel_macro>
-    <xacro:wheel_macro id="2" r_wheel="${r_wheel}" width_wheel="${width_wheel}" collision_factor="8"></xacro:wheel_macro>
-    <xacro:wheel_macro id="3" r_wheel="${r_wheel}" width_wheel="${width_wheel}" collision_factor="8"></xacro:wheel_macro>
+    <xacro:wheel_macro id="left" r_wheel="${r_wheel}" width_wheel="${width_wheel}" collision_factor="8"></xacro:wheel_macro>
+    <xacro:wheel_macro id="right" r_wheel="${r_wheel}" width_wheel="${width_wheel}" collision_factor="8"></xacro:wheel_macro>
+    <xacro:wheel_macro id="back" r_wheel="${r_wheel}" width_wheel="${width_wheel}" collision_factor="8"></xacro:wheel_macro>
     <!-- Joints -->
-    <joint name="steering_1" type="continuous">
+    <joint name="steering_left" type="continuous">
         <parent link="base_link"/>
-        <child link="mod_1"/>
+        <child link="mod_left"/>
+        <origin xyz="${l_wheel/2} ${l_wheel*0.866} 0" rpy="0 0 0"/>
+        <axis xyz="0 0 1"/>
+    </joint>
+    <joint name="steering_right" type="continuous">
+        <parent link="base_link"/>
+        <child link="mod_right"/>
         <origin xyz="${l_wheel/2} ${-l_wheel*0.866} 0" rpy="0 0 0"/>
         <axis xyz="0 0 1"/>
     </joint>
-    <joint name="steering_2" type="continuous">
+    <joint name="steering_back" type="continuous">
         <parent link="base_link"/>
-        <child link="mod_2"/>
-        <origin xyz="${l_wheel/2} ${l_wheel*0.866} 0" rpy="0 0 0"/>
-        <axis xyz="0 0 1"/>
-    </joint>
-    <joint name="steering_3" type="continuous">
-        <parent link="base_link"/>
-        <child link="mod_3"/>
+        <child link="mod_back"/>
         <origin xyz="${-l_wheel} 0 0" rpy="0 0 0"/>
         <axis xyz="0 0 1"/>
     </joint>
-    <joint name="driveshaft_1" type="continuous">
-        <parent link="mod_1"/>
-        <child link="wheel_1"/>
+    <joint name="driveshaft_left" type="continuous">
+        <parent link="mod_left"/>
+        <child link="wheel_left"/>
         <origin xyz="0 0 0" rpy="${90*d2r} 0 0"/>
         <axis xyz="0 0 1"/>
     </joint>
-    <joint name="driveshaft_2" type="continuous">
-        <parent link="mod_2"/>
-        <child link="wheel_2"/>
+    <joint name="driveshaft_right" type="continuous">
+        <parent link="mod_right"/>
+        <child link="wheel_right"/>
         <origin xyz="0 0 0" rpy="${90*d2r} 0 0"/>
         <axis xyz="0 0 1"/>
     </joint>
-    <joint name="driveshaft_3" type="continuous">
-        <parent link="mod_3"/>
-        <child link="wheel_3"/>
+    <joint name="driveshaft_back" type="continuous">
+        <parent link="mod_back"/>
+        <child link="wheel_back"/>
         <origin xyz="0 0 0" rpy="${90*d2r} 0 0"/>
         <axis xyz="0 0 1"/>

File: ghost_sim/urdf/ghost1_sim_base.xacro (robot description, xacro)
@@ -12,10 +12,10 @@
         <plugin name="gazebo_ros_joint_state_publisher" filename="libgazebo_ros_joint_state_publisher.so">
             <update_rate>100</update_rate>
-            <joint_name>steering_1</joint_name>
-            <joint_name>steering_2</joint_name>
-            <joint_name>steering_3</joint_name>
-            <joint_name>driveshaft_1</joint_name>
-            <joint_name>driveshaft_2</joint_name>
-            <joint_name>driveshaft_3</joint_name>
+            <joint_name>steering_left</joint_name>
+            <joint_name>steering_right</joint_name>
+            <joint_name>steering_back</joint_name>
+            <joint_name>driveshaft_left</joint_name>
+            <joint_name>driveshaft_right</joint_name>
+            <joint_name>driveshaft_back</joint_name>
         </plugin>
         <plugin name="swerve_odometry_plugin" filename="libswerve_odometry_plugin.so">

Commit message: updates URDF with dimensions from most recent CAD tweaks URDF colors in RVIZ

File: ghost_description/urdf/ghost1.xacro (robot description, xacro)
@@ -2,5 +2,5 @@
 <robot name="ghost1" xmlns:xacro="http://ros.org/wiki/xacro">
     <xacro:include filename="$(find ghost_description)/urdf/swerve_macros.xacro"/>
-    <xacro:property name="l_wheel" value="0.2286"/> <!-- 9" center to wheel modules-->
+    <xacro:property name="dist_to_wheel" value="0.2286"/> <!-- 9" center to wheel modules-->
     <xacro:property name="r_wheel" value="0.034925"/> <!-- 1.375" wheel radius-->
     <xacro:property name="width_wheel" value="0.0254"/> <!-- 1" wheel width-->
@@ -11,7 +11,9 @@
         <origin xyz="0 0 0" rpy="0 0 0"/>
         <geometry>
-            <sphere radius="${com_radius}"/>
+            <box size="0.0127 0.29 0.0254"/>
         </geometry>
-        <material name="white"/>
+            <material name="silver">
+                <color rgba="0.9 0.9 0.9 1.0"/>
+            </material>
         </visual>
         <!--Inertia estimated for solid cylinder of radius 9" and height 3" with mass 7kg-->
@@ -41,5 +43,56 @@
         <parent link="base_link"/>
         <child link="base_footprint"/>
-        <origin xyz="0 0 ${- r_wheel}" rpy="0 0 0"/>
+        <origin xyz="0 0 -0.052585" rpy="0 0 0"/>
+        <axis xyz="0 0 1"/>
+    </joint>
+    <link name="front_bar">
+        <visual>
+        <origin xyz="0 0 0" rpy="0 0 0"/>
+        <geometry>
+            <box size="0.0127 0.35 0.0254"/>
+        </geometry>
+            <material name="silver">
+                <color rgba="0.9 0.9 0.9 1.0"/>
+            </material>
+        </visual>
+    </link>
+    <joint name="front_bar_joint" type="fixed">
+        <parent link="base_link"/>
+        <child link="front_bar"/>
+        <origin xyz="0.175 0 0" rpy="0 0 0"/>
+        <axis xyz="0 0 1"/>
+    </joint>
+    <link name="left_bar">
+        <visual>
+        <origin xyz="0 0 0" rpy="0 0 0"/>
+        <geometry>
+            <box size="0.0127 0.35 0.0254"/>
+        </geometry>
+            <material name="silver">
+                <color rgba="0.9 0.9 0.9 1.0"/>
+            </material>
+        </visual>
+    </link>
+    <joint name="left_bar_joint" type="fixed">
+        <parent link="base_link"/>
+        <child link="left_bar"/>
+        <origin xyz="-0.05 0.125 0" rpy="0 0 -1.0471"/>
+        <axis xyz="0 0 1"/>
+    </joint>
+    <link name="right_bar">
+        <visual>
+        <origin xyz="0 0 0" rpy="0 0 0"/>
+        <geometry>
+            <box size="0.0127 0.35 0.0254"/>
+        </geometry>
+            <material name="silver">
+                <color rgba="0.9 0.9 0.9 1.0"/>
+            </material>
+    </visual>
+    </link>
+    <joint name="right_bar_joint" type="fixed">
+        <parent link="base_link"/>
+        <child link="right_bar"/>
+        <origin xyz="-0.05 -0.125 0" rpy="0 0 1.0471"/>
         <axis xyz="0 0 1"/>
     </joint>
@@ -56,5 +109,5 @@
         <parent link="base_link"/>
         <child link="mod_left"/>
-        <origin xyz="${l_wheel/2} ${l_wheel*0.866} 0" rpy="0 0 0"/>
+        <origin xyz="0.126365 0.180975 0.0812" rpy="0 0 0"/>
         <axis xyz="0 0 1"/>
     </joint>
@@ -62,5 +115,5 @@
         <parent link="base_link"/>
         <child link="mod_right"/>
-        <origin xyz="${l_wheel/2} ${-l_wheel*0.866} 0" rpy="0 0 0"/>
+        <origin xyz="0.126365 -0.180975 0.0812" rpy="0 0 0"/>
         <axis xyz="0 0 1"/>
     </joint>
@@ -68,5 +121,5 @@
         <parent link="base_link"/>
         <child link="mod_back"/>
-        <origin xyz="${-l_wheel} 0 0" rpy="0 0 0"/>
+        <origin xyz="-0.187 0.0 0.0812" rpy="0 0 0"/>
         <axis xyz="0 0 1"/>
     </joint>
@@ -74,5 +127,5 @@
         <parent link="mod_left"/>
         <child link="wheel_left"/>
-        <origin xyz="0 0 0" rpy="${90*d2r} 0 0"/>
+        <origin xyz="0 0 -0.09886" rpy="${90*d2r} 0 0"/>
         <axis xyz="0 0 1"/>
     </joint>
@@ -80,5 +133,5 @@
         <parent link="mod_right"/>
         <child link="wheel_right"/>
-        <origin xyz="0 0 0" rpy="${90*d2r} 0 0"/>
+        <origin xyz="0 0 -0.09886" rpy="${90*d2r} 0 0"/>
         <axis xyz="0 0 1"/>
     </joint>
@@ -86,5 +139,5 @@
         <parent link="mod_back"/>
         <child link="wheel_back"/>
-        <origin xyz="0 0 0" rpy="${90*d2r} 0 0"/>
+        <origin xyz="0 0 -0.09886" rpy="${90*d2r} 0 0"/>
         <axis xyz="0 0 1"/>
     </joint>
@@ -106,7 +159,7 @@
         <parent link="base_link"/>
         <child link="lidar_link"/>
-        <origin xyz="0 0 0.1" rpy="0 0 0"/>
+        <origin xyz="-0.19015 0 0.2145" rpy="0 0 0"/>
     </joint>
-    <link name="camera_base_link">
+    <!-- <link name="camera_base_link">
         <inertial>
             <origin xyz="0.0 0 0.0" rpy="0 0 0"/>
@@ -118,5 +171,5 @@
         <parent link="base_link"/>
         <child link="camera_base_link"/>
-        <origin xyz="${l_wheel/2} 0 0.33" rpy="0 0 0"/>
+        <origin xyz="${dist_to_wheel/2} 0 0.33" rpy="0 0 0"/>
     </joint>
     <link name="camera_view_link">
@@ -131,4 +184,4 @@
         <child link="camera_view_link"/>
         <origin xyz="0 0 0" rpy="0 0.7853975 0"/>
-    </joint>
+    </joint> -->
 </robot>

File: ghost_description/urdf/swerve_macros.xacro (robot description, xacro)
@@ -12,4 +12,13 @@
                 izz="0.001902"/>
         </inertial>
+        <visual>
+            <origin xyz="0 0 -0.05" rpy="0 0 0"/>
+            <geometry>
+                <cylinder radius="0.04826" length="0.0127"/>
+            </geometry>
+            <material name="silver">
+                <color rgba="0.9 0.9 0.9 1.0"/>
+            </material>
+        </visual>
     </link>
     </xacro:macro>
@@ -21,5 +30,7 @@
                     <cylinder radius="${r_wheel}" length="${width_wheel}"/>
                 </geometry>
-                <material name="black"/>
+                <material name="black">
+                    <color rgba="0 0 0 1.0"/>
+                </material>
             </visual>
             <collision>

Commit message: added cv to rviz

File: ghost_description/urdf/ghost1.xacro (robot description, xacro)
@@ -161,5 +161,5 @@
         <origin xyz="-0.19015 0 0.2145" rpy="0 0 0"/>
     </joint>
-    <!-- <link name="camera_base_link">
+    <link name="camera_base_link">
         <inertial>
             <origin xyz="0.0 0 0.0" rpy="0 0 0"/>
@@ -173,5 +173,5 @@
         <origin xyz="${dist_to_wheel/2} 0 0.33" rpy="0 0 0"/>
     </joint>
-    <link name="camera_view_link">
+    <link name="camera_color_optical_frame">
         <inertial>
             <origin xyz="0.0 0 0.0" rpy="0 0 0"/>
@@ -182,6 +182,6 @@
     <joint name="camera_view_joint" type="fixed">
         <parent link="camera_base_link"/>
-        <child link="camera_view_link"/>
+        <child link="camera_color_optical_frame"/>
         <origin xyz="0 0 0" rpy="0 0.7853975 0"/>
-    </joint> -->
+    </joint>
 </robot>

Commit message: worlds updates 1

File: ghost_description/urdf/ghost1.xacro (robot description, xacro)
@@ -159,5 +159,5 @@
         <parent link="base_link"/>
         <child link="lidar_link"/>
-        <origin xyz="-0.19015 0 0.2145" rpy="0 0 0"/>
+        <origin xyz="-0.19015 0 0.2145" rpy="0 0 ${67.562*d2r}"/>
     </joint>
     <!-- <link name="camera_base_link">

Commit message: PArticle Filter Testing on HArdware

File: ghost_description/urdf/ghost1.xacro (robot description, xacro)
@@ -60,5 +60,5 @@
         <parent link="base_link"/>
         <child link="front_bar"/>
-        <origin xyz="0.175 0 0" rpy="0 0 0"/>
+        <origin xyz="0.156 0 0" rpy="0 0 0"/>
         <axis xyz="0 0 1"/>
     </joint>
@@ -77,5 +77,5 @@
         <parent link="base_link"/>
         <child link="left_bar"/>
-        <origin xyz="-0.05 0.125 0" rpy="0 0 -1.0471"/>
+        <origin xyz="-0.069 0.125 0" rpy="0 0 -1.0471"/>
         <axis xyz="0 0 1"/>
     </joint>
@@ -94,5 +94,5 @@
         <parent link="base_link"/>
         <child link="right_bar"/>
-        <origin xyz="-0.05 -0.125 0" rpy="0 0 1.0471"/>
+        <origin xyz="-0.069 -0.125 0" rpy="0 0 1.0471"/>
         <axis xyz="0 0 1"/>
     </joint>
@@ -109,5 +109,5 @@
         <parent link="base_link"/>
         <child link="mod_left"/>
-        <origin xyz="0.126365 0.180975 0.0812" rpy="0 0 0"/>
+        <origin xyz="0.10452 0.180975 0.0812" rpy="0 0 0"/>
         <axis xyz="0 0 1"/>
     </joint>
@@ -115,5 +115,5 @@
         <parent link="base_link"/>
         <child link="mod_right"/>
-        <origin xyz="0.126365 -0.180975 0.0812" rpy="0 0 0"/>
+        <origin xyz="0.10452 -0.180975 0.0812" rpy="0 0 0"/>
         <axis xyz="0 0 1"/>
     </joint>
@@ -121,5 +121,5 @@
         <parent link="base_link"/>
         <child link="mod_back"/>
-        <origin xyz="-0.187 0.0 0.0812" rpy="0 0 0"/>
+        <origin xyz="-0.209 0.0 0.0812" rpy="0 0 0"/>
         <axis xyz="0 0 1"/>
     </joint>
@@ -159,5 +159,5 @@
         <parent link="base_link"/>
         <child link="lidar_link"/>
-        <origin xyz="-0.19015 0 0.2145" rpy="0 0 ${67.562*d2r}"/>
+        <origin xyz="-0.209 0 0.2145" rpy="0 0 ${67.562*d2r}"/>
     </joint>
     <!-- <link name="camera_base_link">

Commit message: adds joint dynamics to URDF

File: ghost_description/urdf/ghost1.xacro (robot description, xacro)
@@ -110,4 +110,5 @@
         <child link="mod_left"/>
         <origin xyz="0.10452 0.180975 0.0812" rpy="0 0 0"/>
+        <dynamics damping="0.0" friction="0.0"/>
         <axis xyz="0 0 1"/>
     </joint>
@@ -116,4 +117,5 @@
         <child link="mod_right"/>
         <origin xyz="0.10452 -0.180975 0.0812" rpy="0 0 0"/>
+        <dynamics damping="0.0" friction="0.0"/>
         <axis xyz="0 0 1"/>
     </joint>
@@ -122,4 +124,5 @@
         <child link="mod_back"/>
         <origin xyz="-0.209 0.0 0.0812" rpy="0 0 0"/>
+        <dynamics damping="0.0" friction="0.0"/>
         <axis xyz="0 0 1"/>
     </joint>
@@ -128,4 +131,5 @@
         <child link="wheel_left"/>
         <origin xyz="0 0 -0.09886" rpy="${90*d2r} 0 0"/>
+        <dynamics damping="0.0" friction="0.0"/>
         <axis xyz="0 0 1"/>
     </joint>
@@ -134,4 +138,5 @@
         <child link="wheel_right"/>
         <origin xyz="0 0 -0.09886" rpy="${90*d2r} 0 0"/>
+        <dynamics damping="0.0" friction="0.0"/>
         <axis xyz="0 0 1"/>
     </joint>
@@ -140,4 +145,5 @@
         <child link="wheel_back"/>
         <origin xyz="0 0 -0.09886" rpy="${90*d2r} 0 0"/>
+        <dynamics damping="0.0" friction="0.0"/>
         <axis xyz="0 0 1"/>
     </joint>

Commit message: renames swerve joints/links for clarity

File: ghost_description/urdf/ghost1.xacro (robot description, xacro)
@@ -106,42 +106,42 @@
     <xacro:wheel_macro id="back" r_wheel="${r_wheel}" width_wheel="${width_wheel}" collision_factor="8"></xacro:wheel_macro>
     <!-- Joints -->
-    <joint name="steering_left" type="continuous">
+    <joint name="steering_joint_left" type="continuous">
         <parent link="base_link"/>
-        <child link="mod_left"/>
+        <child link="steering_link_left"/>
         <origin xyz="0.10452 0.180975 0.0812" rpy="0 0 0"/>
         <dynamics damping="0.0" friction="0.0"/>
         <axis xyz="0 0 1"/>
     </joint>
-    <joint name="steering_right" type="continuous">
+    <joint name="steering_joint_right" type="continuous">
         <parent link="base_link"/>
-        <child link="mod_right"/>
+        <child link="steering_link_right"/>
         <origin xyz="0.10452 -0.180975 0.0812" rpy="0 0 0"/>
         <dynamics damping="0.0" friction="0.0"/>
         <axis xyz="0 0 1"/>
     </joint>
-    <joint name="steering_back" type="continuous">
+    <joint name="steering_joint_back" type="continuous">
         <parent link="base_link"/>
-        <child link="mod_back"/>
+        <child link="steering_link_back"/>
         <origin xyz="-0.209 0.0 0.0812" rpy="0 0 0"/>
         <dynamics damping="0.0" friction="0.0"/>
         <axis xyz="0 0 1"/>
     </joint>
-    <joint name="driveshaft_left" type="continuous">
-        <parent link="mod_left"/>
-        <child link="wheel_left"/>
+    <joint name="wheel_joint_left" type="continuous">
+        <parent link="steering_link_left"/>
+        <child link="wheel_link_left"/>
         <origin xyz="0 0 -0.09886" rpy="${90*d2r} 0 0"/>
         <dynamics damping="0.0" friction="0.0"/>
         <axis xyz="0 0 1"/>
     </joint>
-    <joint name="driveshaft_right" type="continuous">
-        <parent link="mod_right"/>
-        <child link="wheel_right"/>
+    <joint name="wheel_joint_right" type="continuous">
+        <parent link="steering_link_right"/>
+        <child link="wheel_link_right"/>
         <origin xyz="0 0 -0.09886" rpy="${90*d2r} 0 0"/>
         <dynamics damping="0.0" friction="0.0"/>
         <axis xyz="0 0 1"/>
     </joint>
-    <joint name="driveshaft_back" type="continuous">
-        <parent link="mod_back"/>
-        <child link="wheel_back"/>
+    <joint name="wheel_joint_back" type="continuous">
+        <parent link="steering_link_back"/>
+        <child link="wheel_link_back"/>
         <origin xyz="0 0 -0.09886" rpy="${90*d2r} 0 0"/>
         <dynamics damping="0.0" friction="0.0"/>

File: ghost_description/urdf/swerve_macros.xacro (robot description, xacro)
@@ -3,5 +3,5 @@
     <!-- Steering Module Macro -->
     <xacro:macro name="steering_macro" params="id">
-    <link name="mod_${id}">
+    <link name="steering_link_${id}">
         <inertial>
             <origin xyz="0 0 0" rpy="0 0 0"/>
@@ -25,5 +25,5 @@
     <!-- Wheel Macro -->
     <xacro:macro name="wheel_macro" params="id r_wheel width_wheel collision_factor">
-    <link name="wheel_${id}">
+    <link name="wheel_link_${id}">
             <visual>
                 <geometry>
