Commit message: Swerve moves in sim with pseudo turret. Must validate with plots

File: 03_ROS/ghost_description/urdf/ghost1.xacro (robot description, xacro)
@@ -101,8 +101,10 @@
     <xacro:steering_macro id="right"></xacro:steering_macro>
     <xacro:steering_macro id="back"></xacro:steering_macro>
+    <xacro:steering_macro id="top_test"></xacro:steering_macro>
     <!-- Wheel Modules -->
     <xacro:wheel_macro id="left" r_wheel="${r_wheel}" width_wheel="${width_wheel}" collision_factor="8"></xacro:wheel_macro>
     <xacro:wheel_macro id="right" r_wheel="${r_wheel}" width_wheel="${width_wheel}" collision_factor="8"></xacro:wheel_macro>
     <xacro:wheel_macro id="back" r_wheel="${r_wheel}" width_wheel="${width_wheel}" collision_factor="8"></xacro:wheel_macro>
+    <xacro:wheel_macro id="top_test" r_wheel="${r_wheel}" width_wheel="${width_wheel}" collision_factor="8"></xacro:wheel_macro>
     <!-- Joints -->
     <joint name="steering_joint_left" type="continuous">
@@ -124,4 +126,11 @@
         <child link="steering_link_back"/>
         <origin xyz="-0.209 0.0 0.0812" rpy="0 0 0"/>
+        <dynamics damping="0.0" friction="0.0"/>
+        <axis xyz="0 0 1"/>
+    </joint>
+    <joint name="steering_top_test" type="continuous">
+        <parent link="base_link"/>
+        <child link="steering_link_top_test"/>
+        <origin xyz="0 0 0.0812" rpy="${180*d2r} 0 0"/>
         <dynamics damping="0.0" friction="0.0"/>
         <axis xyz="0 0 1"/>
@@ -147,4 +156,11 @@
         <dynamics damping="0.0" friction="0.0"/>
         <axis xyz="0 0 1"/>
+    </joint>
+    <joint name="wheel_top_test" type="continuous">
+        <parent link="steering_link_top_test"/>
+        <child link="wheel_link_top_test"/>
+        <origin xyz="0 0 -0.09886" rpy="${90*d2r} 0 0"/>
+        <dynamics damping="0.0" friction="0.0"/>
+        <axis xyz="0 0 0"/>
     </joint>
     <!-- Sensors -->

File: 03_ROS/ghost_sim/urdf/ghost1_sim_base.xacro (robot description, xacro)
@@ -6,5 +6,5 @@
     <xacro:include filename="$(find ghost_description)/urdf/ghost1.xacro"/>
     <!-- Add Sensors -->
-    <xacro:lidar_macro link_name="lidar_link" topic_name="scan"></xacro:lidar_macro>
+    <!-- <xacro:lidar_macro link_name="lidar_link" topic_name="scan"></xacro:lidar_macro> -->
     <!-- <xacro:imu_macro parent_link="camera_view_link"></xacro:imu_macro> -->
     <!-- Joint State Publisher -->
@@ -15,7 +15,9 @@
                 steering_joint_right
                 steering_joint_back
+                steering_top_test
                 wheel_joint_left
                 wheel_joint_right
                 wheel_joint_back
+                wheel_top_test
             </joint_names>
             <!-- Motor names must be formatted in this manner in order to index actuator jacobian -->
@@ -56,6 +58,8 @@
             <!-- Width = # Motors, Height = # Joints -->
             <actuator_jacobian>
+              0    0    0    0    0    0    0    0
+              0    0    0    0    0    0    0    0
+              0    0    0    0    0    0    0    0
             1.0    0    0    0    0    0    0    0
-              0    0    0    0    0    0    0    0
               0    0    0    0    0    0    0    0
               0    0    0    0    0    0    0    0
@@ -74,59 +78,8 @@
             0 0 0 0
             0 0 0 0
+            0 0 0 0
+            0 0 0 0
             </sensor_jacobian>
         </plugin>
     </gazebo>
-        <!-- Gazebo Plugins -->
-    <gazebo>
-        <!-- Motor Models -->
-        <!-- 0.05 Steering -->
-        <!-- <xacro:joint_pid_macro
-            joint_name="steering_left"
-            link_name="mod_left"
-            gear_ratio="2.0"
-            position_gain="0.05"
-            vel_gain="0.04"
-            accel_gain="0.0">
-        </xacro:joint_pid_macro> -->
-        <!-- <xacro:joint_pid_macro
-            joint_name="steering_right"
-            link_name="mod_right"
-            gear_ratio="2.0"
-            position_gain="0.05"
-            vel_gain="0.04"
-            accel_gain="0.0">
-        </xacro:joint_pid_macro>
-        <xacro:joint_pid_macro
-            joint_name="steering_back"
-            link_name="mod_back"
-            gear_ratio="2.0"
-            position_gain="0.05"
-            vel_gain="0.04"
-            accel_gain="0.0">
-        </xacro:joint_pid_macro>
-        <xacro:joint_pid_macro
-            joint_name="driveshaft_left"
-            link_name="wheel_left"
-            gear_ratio="5.0"
-            position_gain="0.0"
-            vel_gain="0.04"
-            accel_gain="0.0">
-        </xacro:joint_pid_macro>
-        <xacro:joint_pid_macro
-            joint_name="driveshaft_right"
-            link_name="wheel_right"
-            gear_ratio="5.0"
-            position_gain="0.0"
-            vel_gain="0.04"
-            accel_gain="0.0">
-        </xacro:joint_pid_macro>
-        <xacro:joint_pid_macro
-            joint_name="driveshaft_back"
-            link_name="wheel_back"
-            gear_ratio="5.0"
-            position_gain="0.0"
-            vel_gain="0.04"
-            accel_gain="0.0">
-        </xacro:joint_pid_macro>   -->
-    </gazebo>
 </robot>

Commit message: adds triballs

File: 03_ROS/ghost_description/urdf/ghost1.xacro (robot description, xacro)
@@ -1,4 +1,5 @@
 <?xml version="1.0"?>
 <robot name="ghost1" xmlns:xacro="http://ros.org/wiki/xacro">
+    <origin xyz="1 1 0" rpy="0 0 0"/><!--${pi}-->
     <xacro:include filename="$(find ghost_description)/urdf/swerve_macros.xacro"/>
     <xacro:property name="dist_to_wheel" value="0.2286"/> <!-- 9" center to wheel modules-->
