Commit message: EKF works with test diff drive if given cmd_vel. Need to test EKF when diff drive is stationary. Must be tuned again for swerve drive.

File: 03_ROS/ghost_description/urdf/swerve_macros.xacro (robot description, xacro)
@@ -62,5 +62,5 @@
                 <friction>
                     <torsional>
-                        <coefficient>1.0</coefficient>
+                        <coefficient>0.5</coefficient>
                         <patch_radius>0.01</patch_radius>
                     </torsional>

File: 03_ROS/ghost_sim/urdf/test_tank_init.xacro (robot description, xacro)
@@ -8,11 +8,8 @@
         <plugin name="gazebo_ros_diff_drive" filename="libgazebo_ros_diff_drive.so">
             <!-- Update rate in Hz -->
-            <update_rate>1</update_rate>
+            <update_rate>30.0</update_rate>
             <!-- wheels -->
-            <left_joint>wheel_joint_left_front</left_joint>
-            <left_joint>wheel_joint_left_back</left_joint>
-            <right_joint>wheel_joint_right_front</right_joint>
-            <right_joint>wheel_joint_right_back</right_joint>
-            <num_wheel_pairs>2</num_wheel_pairs>
+            <left_joint>left_wheel_hinge</left_joint>
+            <right_joint>right_wheel_hinge</right_joint>
             <!-- kinematics -->
             <wheel_separation>1.25</wheel_separation>
@@ -24,5 +21,5 @@
             <command_topic>cmd_vel</command_topic>
             <!-- output: odometrySource 0 for ENCODER 1 for WORLD -->
-            <odometrySource>0</odometrySource>
+            <odometrySource>1</odometrySource>
             <publish_odom>true</publish_odom>
             <publish_odom_tf>true</publish_odom_tf>

File: 03_ROS/ghost_sim/urdf/test_tank_sim_base.xacro (robot description, xacro)
@@ -1,151 +1,136 @@
 <?xml version="1.0"?>
 <robot name="test_diff_drive" xmlns:xacro="http://ros.org/wiki/xacro">
-    <xacro:include filename="$(find ghost_description)/urdf/swerve_macros.xacro"/>
-    <xacro:include filename="$(find ghost_sim)/urdf/macros/actuator_macros.xacro"/>
-    <xacro:property name="dist_to_wheel" value="0.2286"/> <!-- 9" center to wheel modules-->
-    <xacro:property name="r_wheel" value="0.034925"/> <!-- 1.375" wheel radius-->
-    <xacro:property name="width_wheel" value="0.0254"/> <!-- 1" wheel width-->
-    <xacro:property name="com_radius" value="0.02"/>
-    <xacro:property name="d2r" value="${3.14159/180}"/>
-    <link name="base_link">
-        <visual>
-            <origin xyz="0 0 0" rpy="0 0 0"/>
+    <xacro:property name='d2r' value="${3.14159/180}"/>
+    <link name='base_link'>
+        <pose>0 0 0.1 0 0 0</pose>
+        <inertial>
+            <mass value="15.0"/>
+            <origin xyz="0.0 0 0.1" rpy=" 0 0 0"/>
+            <inertia
+                ixx="0.1" ixy="0" ixz="0"
+                iyy="0.1" iyz="0"
+                izz="0.1"/>
+        </inertial>
+        <collision name='collision'>
             <geometry>
-                <box size="0.0254 0.29 0.0254"/>
+                <box size=".4 .2 .1"/>
             </geometry>
-                <material name="silver">
-                    <color rgba="0.9 0.9 0.9 1.0"/>
-                </material>
+        </collision>
+        <visual name='chassis_visual'>
+            <origin xyz="0 0 0" rpy=" 0 0 0"/>
+            <geometry>
+                <box size=".4 .2 .1"/>
+            </geometry>
         </visual>
-        <!--Inertia estimated for solid cylinder of radius 9" and height 3" with mass 7kg-->
-        <inertial>
-            <origin xyz="0 0 0" rpy="0 0 0"/>
-            <mass value="10"/>
-            <inertia
-                ixx="0.094839" ixy="0.0" ixz="0.0"
-                iyy="0.094839" iyz="0.0"
-                izz="0.182903"/>
-        </inertial>
-        <gazebo>
-            <maxVel>3.0</maxVel>
-        </gazebo>
-    </link>
-    <link name="base_footprint">
-        <inertial>
-            <origin xyz="0 0 0" rpy="0 0 0"/>
-            <mass value="0.00001"/>
-            <inertia
-                ixx="0.00001" ixy="0.0" ixz="0.0"
-                iyy="0.00001" iyz="0.0"
-                izz="0.00001"/>
-        </inertial>
-    </link>
-    <joint name="base_footprint_joint" type="fixed">
-        <parent link="base_link"/>
-        <child link="base_footprint"/>
-        <origin xyz="0 0 -0.052585" rpy="0 0 0"/>
-        <axis xyz="0 0 1"/>
-    </joint>
-    <link name="left_bar">
-        <visual>
-            <origin xyz="0 -0.125 0" rpy="0 0 ${90*d2r}"/>
+        <collision name='caster_collision'>
+            <origin xyz="-0.15 0 -0.05" rpy=" 0 0 0"/>
             <geometry>
-                <box size="0.0254 0.29 0.0254"/>
+                <sphere radius="0.05"/>
             </geometry>
-                <material name="silver">
-                    <color rgba="0.9 0.9 0.9 1.0"/>
-                </material>
+            <surface>
+                <friction>
+                <ode>
+                    <mu>0</mu>
+                    <mu2>0</mu2>
+                    <slip1>1.0</slip1>
+                    <slip2>1.0</slip2>
+                </ode>
+                </friction>
+            </surface>
+        </collision>
+        <visual name='caster_visual'>
+            <origin xyz="-0.15 0 -0.05" rpy=" 0 0 0"/>
+            <geometry>
+                <sphere radius="0.05"/>
+            </geometry>
+        </visual>
+        <collision name='caster_front_collision'>
+            <origin xyz="0.15 0 -0.05" rpy=" 0 0 0"/>
+            <geometry>
+                <sphere radius="0.05"/>
+            </geometry>
+            <surface>
+                <friction>
+                <ode>
+                    <mu>0</mu>
+                    <mu2>0</mu2>
+                    <slip1>1.0</slip1>
+                    <slip2>1.0</slip2>
+                </ode>
+                </friction>
+            </surface>
+        </collision>
+        <visual name='caster_front_visual'>
+            <origin xyz="0.15 0 -0.05" rpy=" 0 0 0"/>
+            <geometry>
+                <sphere radius="0.05"/>
+            </geometry>
         </visual>
     </link>
-    <joint name="left_bar_joint" type="fixed">
-        <parent link="base_link"/>
-        <child link="left_bar"/>
-        <origin xyz="0 0 0" rpy="0 0 0"/>
-        <axis xyz="0 0 1"/>
-    </joint>
-    <link name="right_bar">
-        <visual>
-            <origin xyz="0 0 0" rpy="0 0 ${90*d2r}"/>
-            <geometry>
-                <box size="0.0254 0.29 0.0254"/>
-            </geometry>
-                <material name="silver">
-                    <color rgba="0.9 0.9 0.9 1.0"/>
-                </material>
-        </visual>
-    </link>
-    <joint name="right_bar_joint" type="fixed">
-        <parent link="base_link"/>
-        <child link="right_bar"/>
-        <origin xyz="0 0.125 0" rpy="0 0 0"/>
-        <axis xyz="0 0 1"/>
-    </joint>
-    <!-- Steering Modules -->
-    <xacro:steering_macro id="left_front"></xacro:steering_macro>
-    <xacro:steering_macro id="left_back"></xacro:steering_macro>
-    <xacro:steering_macro id="right_front"></xacro:steering_macro>
-    <xacro:steering_macro id="right_back"></xacro:steering_macro>
-    <!-- Joints -->
-    <joint name="steering_joint_left_front" type="continuous">
-        <parent link="base_link"/>
-        <child link="steering_link_left_front"/>
-        <origin xyz="0.145 -0.145 0.0812" rpy="0 0 0"/>
-        <dynamics damping="0.0" friction="0.0"/>
-        <axis xyz="0 0 1"/>
-    </joint>
-    <joint name="steering_joint_left_back" type="continuous">
-        <parent link="base_link"/>
-        <child link="steering_link_left_back"/>
-        <origin xyz="-0.145 -0.145 0.0812" rpy="0 0 0"/>
-        <dynamics damping="0.0" friction="0.0"/>
-        <axis xyz="0 0 1"/>
-    </joint>
-    <joint name="steering_joint_right_front" type="continuous">
-        <parent link="base_link"/>
-        <child link="steering_link_right_front"/>
-        <origin xyz="0.145 0.145 0.0812" rpy="0 0 0"/>
-        <dynamics damping="0.0" friction="0.0"/>
-        <axis xyz="0 0 1"/>
-    </joint>
-    <joint name="steering_joint_right_back" type="continuous">
-        <parent link="base_link"/>
-        <child link="steering_link_right_back"/>
-        <origin xyz="-0.145 0.145 0.0812" rpy="0 0 0"/>
-        <dynamics damping="0.0" friction="0.0"/>
-        <axis xyz="0 0 1"/>
-    </joint>
-    <xacro:wheel_macro id="left_front" r_wheel="${r_wheel}" width_wheel="${width_wheel}" collision_factor="8"></xacro:wheel_macro>
-    <xacro:wheel_macro id="left_back" r_wheel="${r_wheel}" width_wheel="${width_wheel}" collision_factor="8"></xacro:wheel_macro>
-    <xacro:wheel_macro id="right_front" r_wheel="${r_wheel}" width_wheel="${width_wheel}" collision_factor="8"></xacro:wheel_macro>
-    <xacro:wheel_macro id="right_back" r_wheel="${r_wheel}" width_wheel="${width_wheel}" collision_factor="8"></xacro:wheel_macro>
-    <joint name="wheel_joint_left_front" type="continuous">
-        <parent link="steering_link_left_front"/>
-        <child link="wheel_link_left_front"/>
-        <origin xyz="0 0 -0.09886" rpy="${90*d2r} 0 0"/>
-        <dynamics damping="0.0" friction="0.0"/>
-        <axis xyz="0 0 1"/>
-    </joint>
-    <joint name="wheel_joint_left_back" type="continuous">
-        <parent link="steering_link_left_back"/>
-        <child link="wheel_link_left_back"/>
-        <origin xyz="0 0 -0.09886" rpy="${90*d2r} 0 0"/>
-        <dynamics damping="0.0" friction="0.0"/>
-        <axis xyz="0 0 1"/>
-    </joint>
-    <joint name="wheel_joint_right_front" type="continuous">
-        <parent link="steering_link_right_front"/>
-        <child link="wheel_link_right_front"/>
-        <origin xyz="0 0 -0.09886" rpy="${90*d2r} 0 0"/>
-        <dynamics damping="0.0" friction="0.0"/>
-        <axis xyz="0 0 1"/>
-    </joint>
-    <joint name="wheel_joint_right_back" type="continuous">
-        <parent link="steering_link_right_back"/>
-        <child link="wheel_link_right_back"/>
-        <origin xyz="0 0 -0.09886" rpy="${90*d2r} 0 0"/>
-        <dynamics damping="0.0" friction="0.0"/>
-        <axis xyz="0 0 1"/>
-    </joint>
-    <!-- Sensors -->
+  <link name="left_wheel">
+    <!--origin xyz="0.1 0.13 0.1" rpy="0 1.5707 1.5707"/-->
+    <collision name="collision">
+      <origin xyz="0 0 0" rpy="0 1.5707 1.5707"/>
+      <geometry>
+        <cylinder radius="0.1" length="0.05"/>
+      </geometry>
+    </collision>
+    <visual name="left_wheel_visual">
+      <origin xyz="0 0 0" rpy="0 1.5707 1.5707"/>
+      <geometry>
+        <cylinder radius="0.1" length="0.05"/>
+      </geometry>
+    </visual>
+    <inertial>
+      <origin xyz="0 0 0" rpy="0 1.5707 1.5707"/>
+      <mass value="5"/>
+      <inertia
+        ixx=".1" ixy="0.0" ixz="0.0"
+        iyy=".1" iyz="0.0"
+        izz=".1"/>
+    </inertial>
+  </link>
+  <link name="right_wheel">
+    <!--origin xyz="0.1 -0.13 0.1" rpy="0 1.5707 1.5707"/-->
+    <collision name="collision">
+      <origin xyz="0 0 0" rpy="0 1.5707 1.5707"/>
+      <geometry>
+        <cylinder radius="0.1" length="0.05"/>
+      </geometry>
+    </collision>
+    <visual name="right_wheel_visual">
+      <origin xyz="0 0 0" rpy="0 1.5707 1.5707"/>
+      <geometry>
+        <cylinder radius="0.1" length="0.05"/>
+      </geometry>
+    </visual>
+    <inertial>
+      <origin xyz="0 0 0" rpy="0 1.5707 1.5707"/>
+      <mass value="5"/>
+      <inertia
+        ixx=".1" ixy="0.0" ixz="0.0"
+        iyy=".1" iyz="0.0"
+        izz=".1"/>
+    </inertial>
+  </link>
+  <joint type="continuous" name="left_wheel_hinge">
+    <origin xyz="0 0.15 0" rpy="0 0 0"/>
+    <!--origin xyz="0.1 0.13 0" rpy="0 1.5707 1.5707"/-->
+    <child link="left_wheel"/>
+    <parent link="base_link"/>
+    <axis xyz="0 1 0" rpy="0 0 0"/>
+    <limit effort="10000" velocity="1000"/>
+    <joint_properties damping="1.0" friction="1.0"/>
+  </joint>
+  <joint type="continuous" name="right_wheel_hinge">
+    <origin xyz="0 -0.15 0" rpy="0 0 0"/>
+    <!--origin xyz="0.1 -0.13 0" rpy="0 1.5707 1.5707"/-->
+    <child link="right_wheel"/>
+    <parent link="base_link"/>
+    <axis xyz="0 1 0" rpy="0 0 0"/>
+    <limit effort="10000" velocity="1000"/>
+    <joint_properties damping="1.0" friction="1.0"/>
+  </joint>
+  <!-- Sensors -->
     <link name="lidar_link">
         <inertial>
@@ -184,3 +169,3 @@
         <origin xyz="-0.209 0 0.2145" rpy="0 0 ${67.562*d2r}"/>
     </joint>
-</robot>
+  </robot>
