Commit message: robot localization node launches need to validate filtered odom output with plotjuggler

File: 03_ROS/ghost_sim/urdf/macros/sensor_macros.xacro (robot description, xacro)
@@ -37,10 +37,10 @@
         </gazebo>
     </xacro:macro>
-    <xacro:macro name="imu_macro" params="parent_link">
+    <xacro:macro name="imu_macro" params="parent_link topic_name">
         <gazebo reference="${parent_link}">
             <sensor name="imu_sensor" type="imu">
             <plugin filename="libgazebo_ros_imu_sensor.so" name="imu_plugin">
                 <ros>
-                <remapping>~/out:=imu</remapping>
+                <remapping>~/out:=${topic_name}</remapping>
                 </ros>
                 <initial_orientation_as_reference>false</initial_orientation_as_reference>

File: 03_ROS/ghost_sim/urdf/test_tank_init.xacro (robot description, xacro)
@@ -1,13 +1,12 @@
 <?xml version="1.0"?>
 <robot name="test_diff_drive" xmlns:xacro="http://ros.org/wiki/xacro">
-    <!-- <xacro:arg name="imu_size" value="0.1"/> -->
-    <xacro:include filename="$(find ghost_sim)/urdf/test_tank_description.xacro"/>
+    <xacro:include filename="$(find ghost_sim)/urdf/test_tank_sim_base.xacro"/>
     <xacro:include filename="$(find ghost_sim)/urdf/macros/sensor_macros.xacro"/>
     <xacro:lidar_macro link_name="lidar_link" topic_name="scan"></xacro:lidar_macro>
-    <xacro:imu_macro parent_link="camera_view_link"></xacro:imu_macro>
+    <xacro:imu_macro parent_link="base_link" topic_name="imu"></xacro:imu_macro>
     <gazebo>
         <plugin name="gazebo_ros_diff_drive" filename="libgazebo_ros_diff_drive.so">
             <!-- Update rate in Hz -->
-            <update_rate>50</update_rate>
+            <update_rate>1</update_rate>
             <!-- wheels -->
             <left_joint>wheel_joint_left_front</left_joint>
@@ -24,7 +23,8 @@
             <!-- input -->
             <command_topic>cmd_vel</command_topic>
-            <!-- output -->
-            <publish_odom>false</publish_odom>
-            <publish_odom_tf>false</publish_odom_tf>
+            <!-- output: odometrySource 0 for ENCODER 1 for WORLD -->
+            <odometrySource>0</odometrySource>
+            <publish_odom>true</publish_odom>
+            <publish_odom_tf>true</publish_odom_tf>
             <publish_wheel_tf>true</publish_wheel_tf>
             <odometry_topic>odom</odometry_topic>

File: 03_ROS/ghost_sim/urdf/test_tank_sim_base.xacro (robot description, xacro)
@@ -147,3 +147,40 @@
         <axis xyz="0 0 1"/>
     </joint>
+    <!-- Sensors -->
+    <link name="lidar_link">
+        <inertial>
+            <origin xyz="0.0 0 0.0" rpy="0 0 0"/>
+            <mass value="0.125"/>
+            <inertia ixx="0.001"  ixy="0"  ixz="0" iyy="0.001" iyz="0" izz="0.001" />
+        </inertial>
+        <visual>
+            <origin xyz="0 0 0" rpy="0 0 0"/>
+            <geometry>
+            <cylinder radius="${0.06985/2}" length="0.0254"/>
+            </geometry>
+        </visual>
+    </link>
+    <joint name="lidar_joint" type="fixed">
+        <parent link="base_link"/>
+        <child link="lidar_link"/>
+        <origin xyz="-0.209 0 0.2145" rpy="0 0 ${67.562*d2r}"/>
+    </joint>
+    <link name="imu_link">
+        <inertial>
+            <origin xyz="0.0 0 0.0" rpy="0 0 0"/>
+            <mass value="0.125"/>
+            <inertia ixx="0.001"  ixy="0"  ixz="0" iyy="0.001" iyz="0" izz="0.001" />
+        </inertial>
+        <visual>
+            <origin xyz="0 0 0" rpy="0 0 0"/>
+            <geometry>
+            <cylinder radius="${0.06985/2}" length="0.0254"/>
+            </geometry>
+        </visual>
+    </link>
+    <joint name="imu_joint" type="fixed">
+        <parent link="base_link"/>
+        <child link="imu_link"/>
+        <origin xyz="-0.209 0 0.2145" rpy="0 0 ${67.562*d2r}"/>
+    </joint>
 </robot>
