Commit message: revert swerve changes

File: 11_Robots/ghost_over_under/urdf/ghost1.xacro (robot description, xacro)
@@ -101,10 +101,8 @@
     <xacro:steering_macro id="right"></xacro:steering_macro>
     <xacro:steering_macro id="back"></xacro:steering_macro>
-    <xacro:steering_macro id="top_test"></xacro:steering_macro>
     <!-- Wheel Modules -->
     <xacro:wheel_macro id="left" r_wheel="${r_wheel}" width_wheel="${width_wheel}" collision_factor="8"></xacro:wheel_macro>
     <xacro:wheel_macro id="right" r_wheel="${r_wheel}" width_wheel="${width_wheel}" collision_factor="8"></xacro:wheel_macro>
     <xacro:wheel_macro id="back" r_wheel="${r_wheel}" width_wheel="${width_wheel}" collision_factor="8"></xacro:wheel_macro>
-    <xacro:wheel_macro id="top_test" r_wheel="${r_wheel}" width_wheel="${width_wheel}" collision_factor="8"></xacro:wheel_macro>
     <!-- Joints -->
     <joint name="steering_joint_left" type="continuous">
@@ -126,11 +124,4 @@
         <child link="steering_link_back"/>
         <origin xyz="-0.209 0.0 0.0812" rpy="0 0 0"/>
-        <dynamics damping="0.0" friction="0.0"/>
-        <axis xyz="0 0 1"/>
-    </joint>
-    <joint name="steering_top_test" type="continuous">
-        <parent link="base_link"/>
-        <child link="steering_link_top_test"/>
-        <origin xyz="0 0 0.0812" rpy="${180*d2r} 0 0"/>
         <dynamics damping="0.0" friction="0.0"/>
         <axis xyz="0 0 1"/>
@@ -156,11 +147,4 @@
         <dynamics damping="0.0" friction="0.0"/>
         <axis xyz="0 0 1"/>
-    </joint>
-    <joint name="wheel_top_test" type="continuous">
-        <parent link="steering_link_top_test"/>
-        <child link="wheel_link_top_test"/>
-        <origin xyz="0 0 -0.09886" rpy="${90*d2r} 0 0"/>
-        <dynamics damping="0.0" friction="0.0"/>
-        <axis xyz="0 0 0"/>
     </joint>
     <!-- Sensors -->

File: 11_Robots/ghost_swerve/urdf/swerve_macros.xacro (robot description, xacro)
@@ -62,5 +62,5 @@
                 <friction>
                     <torsional>
-                        <coefficient>0.5</coefficient>
+                        <coefficient>1.0</coefficient>
                         <patch_radius>0.01</patch_radius>
                     </torsional>
