Commit message: fixes typo where front left and back right wheels were switched in URDF

File: 11_Robots/ghost_over_under/urdf/ghost_15.xacro (robot description, xacro)
@@ -98,66 +98,66 @@
     </joint>
     <!-- Steering Modules -->
-    <xacro:steering_macro id="frontleft"></xacro:steering_macro>
-    <xacro:steering_macro id="frontright"></xacro:steering_macro>
-    <xacro:steering_macro id="backleft"></xacro:steering_macro>
-    <xacro:steering_macro id="backright"></xacro:steering_macro>
+    <xacro:steering_macro id="front_left"></xacro:steering_macro>
+    <xacro:steering_macro id="front_right"></xacro:steering_macro>
+    <xacro:steering_macro id="back_left"></xacro:steering_macro>
+    <xacro:steering_macro id="back_right"></xacro:steering_macro>
     <!-- Wheel Modules -->
-    <xacro:wheel_macro id="frontleft" r_wheel="${r_wheel}" width_wheel="${width_wheel}" collision_factor="8"></xacro:wheel_macro>
-    <xacro:wheel_macro id="frontright" r_wheel="${r_wheel}" width_wheel="${width_wheel}" collision_factor="8"></xacro:wheel_macro>
-    <xacro:wheel_macro id="backleft" r_wheel="${r_wheel}" width_wheel="${width_wheel}" collision_factor="8"></xacro:wheel_macro>
-    <xacro:wheel_macro id="backright" r_wheel="${r_wheel}" width_wheel="${width_wheel}" collision_factor="8"></xacro:wheel_macro>
+    <xacro:wheel_macro id="front_left" r_wheel="${r_wheel}" width_wheel="${width_wheel}" collision_factor="8"></xacro:wheel_macro>
+    <xacro:wheel_macro id="front_right" r_wheel="${r_wheel}" width_wheel="${width_wheel}" collision_factor="8"></xacro:wheel_macro>
+    <xacro:wheel_macro id="back_left" r_wheel="${r_wheel}" width_wheel="${width_wheel}" collision_factor="8"></xacro:wheel_macro>
+    <xacro:wheel_macro id="back_right" r_wheel="${r_wheel}" width_wheel="${width_wheel}" collision_factor="8"></xacro:wheel_macro>
     <!-- Joints -->
-    <joint name="steering_joint_backleft" type="continuous">
-        <parent link="base_link"/>
-        <child link="steering_link_backleft"/>
+    <joint name="steering_joint_back_left" type="continuous">
+        <parent link="base_link"/>
+        <child link="steering_link_back_left"/>
         <origin xyz="-0.1143 0.1143 0.0762" rpy="0 0 0"/>
         <dynamics damping="0.0" friction="0.0"/>
         <axis xyz="0 0 1"/>
     </joint>
-    <joint name="steering_joint_backright" type="continuous">
-        <parent link="base_link"/>
-        <child link="steering_link_backright"/>
+    <joint name="steering_joint_back_right" type="continuous">
+        <parent link="base_link"/>
+        <child link="steering_link_back_right"/>
+        <origin xyz="-0.1143 -0.1143 0.0762" rpy="0 0 0"/>
+        <dynamics damping="0.0" friction="0.0"/>
+        <axis xyz="0 0 1"/>
+    </joint>
+    <joint name="steering_joint_front_left" type="continuous">
+        <parent link="base_link"/>
+        <child link="steering_link_front_left"/>
         <origin xyz="0.1143 0.1143 0.0762" rpy="0 0 0"/>
         <dynamics damping="0.0" friction="0.0"/>
         <axis xyz="0 0 1"/>
     </joint>
-    <joint name="steering_joint_frontleft" type="continuous">
-        <parent link="base_link"/>
-        <child link="steering_link_frontleft"/>
-        <origin xyz="-0.1143 -0.1143 0.0762" rpy="0 0 0"/>
-        <dynamics damping="0.0" friction="0.0"/>
-        <axis xyz="0 0 1"/>
-    </joint>
-    <joint name="steering_joint_frontright" type="continuous">
-        <parent link="base_link"/>
-        <child link="steering_link_frontright"/>
+    <joint name="steering_joint_front_right" type="continuous">
+        <parent link="base_link"/>
+        <child link="steering_link_front_right"/>
         <origin xyz="0.1143 -0.1143 0.0762 " rpy="0 0 0"/>
         <dynamics damping="0.0" friction="0.0"/>
         <axis xyz="0 0 1"/>
     </joint>
-    <joint name="wheel_joint_backleft" type="continuous">
-        <parent link="steering_link_backleft"/>
-        <child link="wheel_link_backleft"/>
-        <origin xyz="0 0 -0.09886" rpy="${90*d2r} 0 0"/>
-        <dynamics damping="0.0" friction="0.0"/>
-        <axis xyz="0 0 1"/>
-    </joint>
-    <joint name="wheel_joint_backright" type="continuous">
-        <parent link="steering_link_backright"/>
-        <child link="wheel_link_backright"/>
-        <origin xyz="0 0 -0.09886" rpy="${90*d2r} 0 0"/>
-        <dynamics damping="0.0" friction="0.0"/>
-        <axis xyz="0 0 1"/>
-    </joint>
-    <joint name="wheel_joint_frontleft" type="continuous">
-        <parent link="steering_link_frontleft"/>
-        <child link="wheel_link_frontleft"/>
-        <origin xyz="0 0 -0.09886" rpy="${90*d2r} 0 0"/>
-        <dynamics damping="0.0" friction="0.0"/>
-        <axis xyz="0 0 1"/>
-    </joint>
-    <joint name="wheel_joint_frontright" type="continuous">
-        <parent link="steering_link_frontright"/>
-        <child link="wheel_link_frontright"/>
+    <joint name="wheel_joint_back_left" type="continuous">
+        <parent link="steering_link_back_left"/>
+        <child link="wheel_link_back_left"/>
+        <origin xyz="0 0 -0.09886" rpy="${90*d2r} 0 0"/>
+        <dynamics damping="0.0" friction="0.0"/>
+        <axis xyz="0 0 1"/>
+    </joint>
+    <joint name="wheel_joint_back_right" type="continuous">
+        <parent link="steering_link_back_right"/>
+        <child link="wheel_link_back_right"/>
+        <origin xyz="0 0 -0.09886" rpy="${90*d2r} 0 0"/>
+        <dynamics damping="0.0" friction="0.0"/>
+        <axis xyz="0 0 1"/>
+    </joint>
+    <joint name="wheel_joint_front_left" type="continuous">
+        <parent link="steering_link_front_left"/>
+        <child link="wheel_link_front_left"/>
+        <origin xyz="0 0 -0.09886" rpy="${90*d2r} 0 0"/>
+        <dynamics damping="0.0" friction="0.0"/>
+        <axis xyz="0 0 1"/>
+    </joint>
+    <joint name="wheel_joint_front_right" type="continuous">
+        <parent link="steering_link_front_right"/>
+        <child link="wheel_link_front_right"/>
         <origin xyz="0 0 -0.09886" rpy="${90*d2r} 0 0"/>
         <dynamics damping="0.0" friction="0.0"/>

Commit message: inverts wheel directions in urdf

File: 11_Robots/ghost_over_under/urdf/ghost_15.xacro (robot description, xacro)
@@ -139,5 +139,5 @@
         <parent link="steering_link_back_left"/>
         <child link="wheel_link_back_left"/>
-        <origin xyz="0 0 -0.09886" rpy="${90*d2r} 0 0"/>
+        <origin xyz="0 0 -0.09886" rpy="${-90*d2r} 0 0"/>
         <dynamics damping="0.0" friction="0.0"/>
         <axis xyz="0 0 1"/>
@@ -146,5 +146,5 @@
         <parent link="steering_link_back_right"/>
         <child link="wheel_link_back_right"/>
-        <origin xyz="0 0 -0.09886" rpy="${90*d2r} 0 0"/>
+        <origin xyz="0 0 -0.09886" rpy="${-90*d2r} 0 0"/>
         <dynamics damping="0.0" friction="0.0"/>
         <axis xyz="0 0 1"/>
@@ -153,5 +153,5 @@
         <parent link="steering_link_front_left"/>
         <child link="wheel_link_front_left"/>
-        <origin xyz="0 0 -0.09886" rpy="${90*d2r} 0 0"/>
+        <origin xyz="0 0 -0.09886" rpy="${-90*d2r} 0 0"/>
         <dynamics damping="0.0" friction="0.0"/>
         <axis xyz="0 0 1"/>
@@ -160,5 +160,5 @@
         <parent link="steering_link_front_right"/>
         <child link="wheel_link_front_right"/>
-        <origin xyz="0 0 -0.09886" rpy="${90*d2r} 0 0"/>
+        <origin xyz="0 0 -0.09886" rpy="${-90*d2r} 0 0"/>
         <dynamics damping="0.0" friction="0.0"/>
         <axis xyz="0 0 1"/>

Commit message: enables lidar on hardware fixes lidar tf in URDF

File: 11_Robots/ghost_over_under/urdf/ghost_15.xacro (robot description, xacro)
@@ -254,5 +254,5 @@
         <parent link="base_link"/>
         <child link="lidar_link"/>
-        <origin xyz="-0.1143 -0.1143 0.2921" rpy="0 0 0"/> <!--${67.562*d2r}-->
+        <origin xyz="-0.1143 -0.1143 0.2921" rpy="0 0 ${90.0*d2r}"/>
     </joint>
 </robot>

Commit message: Adds robot state publisher to hardware launch

File: 11_Robots/ghost_over_under/urdf/ghost_15.xacro (robot description, xacro)
@@ -256,3 +256,21 @@
         <origin xyz="-0.1143 -0.1143 0.2921" rpy="0 0 0"/> <!--${67.562*d2r}-->
     </joint>
+    <link name="imu_link">
+        <inertial>
+            <origin xyz="0.0 0 0.0" rpy="0 0 0"/>
+            <mass value="0.125"/>
+            <inertia ixx="0.001"  ixy="0"  ixz="0" iyy="0.001" iyz="0" izz="0.001" />
+        </inertial>
+        <visual>
+            <origin xyz="0 0 0" rpy="0 0 0"/>
+            <geometry>
+            <cylinder radius="${0.06985/2}" length="0.0254"/>
+            </geometry>
+        </visual>
+    </link>
+    <joint name="imu_joint" type="fixed">
+        <parent link="base_link"/>
+        <child link="imu_link"/>
+        <origin xyz="-0.209 0 0.2145" rpy="0 0 ${67.562*d2r}"/>
+    </joint>
 </robot>
