Commit message: Refactors sim stack after hardware refactor

File: 03_ROS/ghost_sim/urdf/test_tank_init.xacro (robot description, xacro)
@@ -3,5 +3,5 @@
     <xacro:include filename="$(find ghost_sim)/urdf/test_tank_sim_base.xacro"/>
     <xacro:include filename="$(find ghost_sim)/urdf/macros/sensor_macros.xacro"/>
-    <xacro:lidar_macro link_name="lidar_link" topic_name="scan"></xacro:lidar_macro>
+    <!-- <xacro:lidar_macro link_name="lidar_link" topic_name="scan"></xacro:lidar_macro> -->
     <xacro:imu_macro parent_link="base_link" topic_name="imu"></xacro:imu_macro>
     <gazebo>

File: 03_ROS/ghost_sim/urdf/test_tank_sim_base.xacro (robot description, xacro)
@@ -133,5 +133,5 @@
   </joint>
   <!-- Sensors -->
-    <link name="lidar_link">
+    <!-- <link name="lidar_link">
         <inertial>
             <origin xyz="0.0 0 0.0" rpy="0 0 0"/>
@@ -150,5 +150,5 @@
         <child link="lidar_link"/>
         <origin xyz="-0.209 0 0.2145" rpy="0 0 ${67.562*d2r}"/>
-    </joint>
+    </joint> -->
     <link name="imu_link">
         <inertial>

Commit message: PF visuals load into RVIZ

File: 03_ROS/ghost_sim/urdf/test_tank_init.xacro (robot description, xacro)
@@ -3,5 +3,5 @@
     <xacro:include filename="$(find ghost_sim)/urdf/test_tank_sim_base.xacro"/>
     <xacro:include filename="$(find ghost_sim)/urdf/macros/sensor_macros.xacro"/>
-    <!-- <xacro:lidar_macro link_name="lidar_link" topic_name="scan"></xacro:lidar_macro> -->
+    <xacro:lidar_macro link_name="lidar_link" topic_name="scan"></xacro:lidar_macro>
     <xacro:imu_macro parent_link="base_link" topic_name="imu"></xacro:imu_macro>
     <gazebo>

File: 03_ROS/ghost_sim/urdf/test_tank_sim_base.xacro (robot description, xacro)
@@ -133,5 +133,5 @@
   </joint>
   <!-- Sensors -->
-    <!-- <link name="lidar_link">
+    <link name="lidar_link">
         <inertial>
             <origin xyz="0.0 0 0.0" rpy="0 0 0"/>
@@ -149,6 +149,6 @@
         <parent link="base_link"/>
         <child link="lidar_link"/>
-        <origin xyz="-0.209 0 0.2145" rpy="0 0 ${67.562*d2r}"/>
-    </joint> -->
+        <origin xyz="-0.209 0 0.180" rpy="0 0 ${67.562*d2r}"/>
+    </joint>
     <link name="imu_link">
         <inertial>
