Commit message: update world file to sdf version 1.7 readded gazebo_ros node fixed bug where base link had no inertia

File: 11_Robots/ghost_high_stakes/urdf/tankbot.xacro (robot description, xacro)
@@ -12,4 +12,12 @@
      </material>
      <link name="base_link">
+      <inertial>
+        <origin xyz="0 0 0" rpy="0 0 0"/>
+        <mass value="5"/>
+        <inertia
+          ixx="0.105847" ixy="0.0" ixz="0.0"
+          iyy="0.105847" iyz="0.0"
+          izz="0.090726"/>
+      </inertial>
       <visual>
       <origin xyz="0 0 0" rpy="0 0 0" />
