Commit message: Adds gazebo tank drive with friction

File: 11_Robots/ghost_high_stakes/urdf/tank_macros.xacro (robot description, xacro)
@@ -2,5 +2,5 @@
 <robot xmlns:xacro="http://www.ros.org/wiki/xacro">
     <!-- Wheel Macro -->
-    <xacro:macro name="wheel_macro" params="id r_wheel width_wheel collision_factor roller_radius roller_width">
+    <xacro:macro name="wheel_macro" params="id r_wheel width_wheel collision_factor">
     <link name="wheel_link_${id}">
             <visual>
@@ -12,104 +12,4 @@
                 </material>
             </visual>
-        <!-- Roller 1 -->
-        <visual>
-            <origin xyz="${r_wheel} 0 0" rpy="0 0 0"/>
-            <geometry>
-                <cylinder radius="${roller_radius}" length="${roller_width}"/>
-            </geometry>
-            <material name="grey">
-                <color rgba="0.5 0.5 0.5 1.0"/>
-            </material>
-        </visual>
-        <!-- Roller 2 -->
-        <visual>
-            <origin xyz="${r_wheel * cos(0.628319)} ${r_wheel * sin(0.628319)} 0" rpy="0 0 0.628319"/>
-            <geometry>
-                <cylinder radius="${roller_radius}" length="${roller_width}"/>
-            </geometry>
-            <material name="grey">
-                <color rgba="0.5 0.5 0.5 1.0"/>
-            </material>
-        </visual>
-        <!-- Roller 3 -->
-        <visual>
-            <origin xyz="${r_wheel * cos(1.25664)} ${r_wheel * sin(1.25664)} 0" rpy="0 0 1.25664"/>
-            <geometry>
-                <cylinder radius="${roller_radius}" length="${roller_width}"/>
-            </geometry>
-            <material name="grey">
-                <color rgba="0.5 0.5 0.5 1.0"/>
-            </material>
-        </visual>
-        <!-- Roller 4 -->
-        <visual>
-            <origin xyz="${r_wheel * cos(1.88496)} ${r_wheel * sin(1.88496)} 0" rpy="0 0 1.88496"/>
-            <geometry>
-                <cylinder radius="${roller_radius}" length="${roller_width}"/>
-            </geometry>
-            <material name="grey">
-                <color rgba="0.5 0.5 0.5 1.0"/>
-            </material>
-        </visual>
-        <!-- Roller 5 -->
-        <visual>
-            <origin xyz="${r_wheel * cos(2.51327)} ${r_wheel * sin(2.51327)} 0" rpy="0 0 2.51327"/>
-            <geometry>
-                <cylinder radius="${roller_radius}" length="${roller_width}"/>
-            </geometry>
-            <material name="grey">
-                <color rgba="0.5 0.5 0.5 1.0"/>
-            </material>
-        </visual>
-                <!-- Roller 6 -->
-        <visual>
-            <origin xyz="${r_wheel * cos(3.14159)} ${r_wheel * sin(3.14159)} 0" rpy="0 0 3.14159"/>
-            <geometry>
-                <cylinder radius="${roller_radius}" length="${roller_width}"/>
-            </geometry>
-            <material name="grey">
-                <color rgba="0.5 0.5 0.5 1.0"/>
-            </material>
-        </visual>
-                <!-- Roller 7 -->
-        <visual>
-            <origin xyz="${r_wheel * cos(3.76991)} ${r_wheel * sin(3.76991)} 0" rpy="0 0 3.76991"/>
-            <geometry>
-                <cylinder radius="${roller_radius}" length="${roller_width}"/>
-            </geometry>
-            <material name="grey">
-                <color rgba="0.5 0.5 0.5 1.0"/>
-            </material>
-        </visual>
-                <!-- Roller 8 -->
-        <visual>
-            <origin xyz="${r_wheel * cos(4.39823)} ${r_wheel * sin(4.39823)} 0" rpy="0 0 4.39823"/>
-            <geometry>
-                <cylinder radius="${roller_radius}" length="${roller_width}"/>
-            </geometry>
-            <material name="grey">
-                <color rgba="0.5 0.5 0.5 1.0"/>
-            </material>
-        </visual>
-                <!-- Roller 9 -->
-        <visual>
-            <origin xyz="${r_wheel * cos(5.02655)} ${r_wheel * sin(5.02655)} 0" rpy="0 0 5.02655"/>
-            <geometry>
-                <cylinder radius="${roller_radius}" length="${roller_width}"/>
-            </geometry>
-            <material name="grey">
-                <color rgba="0.5 0.5 0.5 1.0"/>
-            </material>
-        </visual>
-                <!-- Roller 10 -->
-        <visual>
-            <origin xyz="${r_wheel * cos(5.65487)} ${r_wheel * sin(5.65487)} 0" rpy="0 0 5.65487"/>
-            <geometry>
-                <cylinder radius="${roller_radius}" length="${roller_width}"/>
-            </geometry>
-            <material name="grey">
-                <color rgba="0.5 0.5 0.5 1.0"/>
-            </material>
-        </visual>
             <collision>
                 <origin xyz="0 0 0" rpy="0 0 0"/>
@@ -117,4 +17,12 @@
                     <cylinder radius="${r_wheel}" length="${width_wheel/collision_factor}"/>
                 </geometry>
+          <surface>
+        <friction>
+          <ode>
+         <mu>0.01</mu>
+            <mu2>1.0</mu2>
+          </ode>
+        </friction>
+      </surface>
             </collision>
             <!--Inertia estimated for solid cylinder of radius 2.5" and height 1" with mass 1 lb-->
@@ -148,4 +56,29 @@
         <material>Gazebo/White</material>
     </gazebo>
+    <gazebo reference="wheel_link_${id}">
+        <collision>
+            <origin xyz="0 0 0" rpy="0 0 0"/>
+            <geometry>
+                <cylinder>
+                    <radius>${r_wheel}</radius>
+                    <length>${width_wheel/collision_factor}</length>
+                </cylinder>
+            </geometry>
+            <surface>
+                <friction>
+          <ode>
+        <mu>0.5</mu>
+        <mu2>0.01</mu2>
+        <fdir1>1 0 0</fdir1>
+          </ode>
+                    <!-- <torsional>
+                        <coefficient>1.0</coefficient>
+                        <patch_radius>0.01</patch_radius>
+                    </torsional> -->
+                </friction>
+            </surface>
+        </collision>
+        <material>Gazebo/White</material>
+    </gazebo>
     </xacro:macro>
 </robot>

File: 11_Robots/ghost_high_stakes/urdf/tankbot.xacro (robot description, xacro)
@@ -11,21 +11,39 @@
         <color rgba="1 1 1 1"/>
      </material>
-     <link name="base_link">
-      <inertial>
-        <origin xyz="0 0 0" rpy="0 0 0"/>
-        <mass value="5"/>
-        <inertia
-          ixx="0.105847" ixy="0.0" ixz="0.0"
-          iyy="0.105847" iyz="0.0"
-          izz="0.090726"/>
-      </inertial>
-      <visual>
-      <origin xyz="0 0 0" rpy="0 0 0" />
-         <geometry>
-           <box size= "0 0 0" />
-         </geometry>
-         <material name="white"/>
-       </visual>
-     </link>
+    <link name="base_link">
+        <visual>
+        <origin xyz="0 0 0" rpy="0 0 0"/>
+        <geometry>
+            <box size="0 0 0"/>
+        </geometry>
+            <material name="silver">
+                <color rgba="0.9 0.9 0.9 1.0"/>
+            </material>
+        </visual>
+        <collision>
+        <geometry>
+            <box size="0 0 0"/>
+        </geometry>
+          <surface>
+        <friction>
+          <ode>
+         <mu>0.01</mu>
+            <mu2>1.0</mu2>
+          </ode>
+        </friction>
+      </surface>
+        </collision>
+        <inertial>
+            <origin xyz="0 0 0" rpy="0 0 0"/>
+            <mass value="5"/>
+            <inertia
+                ixx="0.0" ixy="0.0" ixz="0.0"
+                iyy="0.094839" iyz="0.0"
+                izz="0.182903"/>
+        </inertial>
+        <gazebo>
+            <maxVel>3.0</maxVel>
+        </gazebo>
+    </link>
      <link name="back_bar">
         <visual>
@@ -38,4 +56,15 @@
             </material>
         </visual>
+        <inertial>
+            <origin xyz="0 0 0" rpy="0 0 0"/>
+            <mass value="10"/>
+            <inertia
+                ixx="0.0914" ixy="0.0" ixz="0.0"
+                iyy="0.000672" iyz="0.0"
+                izz="0.0910"/>
+        </inertial>
+        <gazebo>
+            <maxVel>3.0</maxVel>
+        </gazebo>
     </link>
     <joint name="back_bar_joint" type="fixed">
@@ -55,4 +84,15 @@
             </material>
         </visual>
+        <inertial>
+            <origin xyz="0 0 0" rpy="0 0 0"/>
+            <mass value="10"/>
+            <inertia
+                ixx="0.0914" ixy="0.0" ixz="0.0"
+                iyy="0.000672" iyz="0.0"
+                izz="0.0910"/>
+        </inertial>
+        <gazebo>
+            <maxVel>3.0</maxVel>
+        </gazebo>
     </link>
     <joint name="left_bar_joint" type="fixed">
@@ -72,4 +112,15 @@
             </material>
     </visual>
+        <inertial>
+            <origin xyz="0 0 0" rpy="0 0 0"/>
+            <mass value="10"/>
+            <inertia
+                ixx="0.0914" ixy="0.0" ixz="0.0"
+                iyy="0.000672" iyz="0.0"
+                izz="0.0910"/>
+        </inertial>
+        <gazebo>
+            <maxVel>3.0</maxVel>
+        </gazebo>
     </link>
     <joint name="right_bar_joint" type="fixed">
@@ -80,51 +131,115 @@
     </joint>
  <!--Wheel Modules-->
-    <xacro:wheel_macro id="front_left" r_wheel="${r_wheel}" width_wheel="${width_wheel}"  roller_width="${roller_width}" roller_radius="${roller_radius}" collision_factor="8"></xacro:wheel_macro>
-    <xacro:wheel_macro id="front_right" r_wheel="${r_wheel}" width_wheel="${width_wheel}"  roller_width="${roller_width}" roller_radius="${roller_radius}" collision_factor="8"></xacro:wheel_macro>
-    <xacro:wheel_macro id="back_left" r_wheel="${r_wheel}" width_wheel="${width_wheel}" roller_width="${roller_width}" roller_radius="${roller_radius}" collision_factor="8"></xacro:wheel_macro>
-    <xacro:wheel_macro id="back_right" r_wheel="${r_wheel}" width_wheel="${width_wheel}"  roller_width="${roller_width}" roller_radius="${roller_radius}" collision_factor="8"></xacro:wheel_macro>
-    <xacro:wheel_macro id="middle_left" r_wheel="${r_wheel}" width_wheel="${width_wheel}"  roller_width="${roller_width}" roller_radius="${roller_radius}" collision_factor="8"></xacro:wheel_macro>
-    <xacro:wheel_macro id="middle_right" r_wheel="${r_wheel}" width_wheel="${width_wheel}"  roller_width="${roller_width}" roller_radius="${roller_radius}" collision_factor="8"></xacro:wheel_macro>
-    <joint name="wheel_joint_back_left" type="continuous">
+    <xacro:wheel_macro id="front_left" r_wheel="${r_wheel}" width_wheel="${width_wheel}"   collision_factor="8"></xacro:wheel_macro>
+    <xacro:wheel_macro id="front_right" r_wheel="${r_wheel}" width_wheel="${width_wheel}"  collision_factor="8"></xacro:wheel_macro>
+    <xacro:wheel_macro id="back_left" r_wheel="${r_wheel}" width_wheel="${width_wheel}"  collision_factor="8"></xacro:wheel_macro>
+    <xacro:wheel_macro id="back_right" r_wheel="${r_wheel}" width_wheel="${width_wheel}"   collision_factor="8"></xacro:wheel_macro>
+    <xacro:wheel_macro id="middle_left" r_wheel="${r_wheel}" width_wheel="${width_wheel}"   collision_factor="8"></xacro:wheel_macro>
+    <xacro:wheel_macro id="middle_right" r_wheel="${r_wheel}" width_wheel="${width_wheel}"   collision_factor="8"></xacro:wheel_macro>
+    <joint name="wheel_joint_back_left" type="fixed">
         <parent link="left_bar"/>
         <child link="wheel_link_back_left"/>
         <origin xyz="-0.0254 -0.10795 0" rpy="${-90*d2r} 0 ${90*d2r}"/>
-        <dynamics damping="0.0" friction="0.0"/>
-        <axis xyz="0 0 1"/>
-    </joint>
-    <joint name="wheel_joint_back_right" type="continuous">
+        <!-- <dynamics damping="0.0" friction="0.0"/> -->
+        <axis xyz="0 0 1"/>
+    </joint>
+    <joint name="wheel_joint_back_right" type="fixed">
         <parent link="right_bar"/>
         <child link="wheel_link_back_right"/>
         <origin xyz="0.0254 -0.10795 0" rpy="${-90*d2r} 0 ${90*d2r}"/>
-        <dynamics damping="0.0" friction="0.0"/>
-        <axis xyz="0 0 1"/>
-    </joint>
-    <joint name="wheel_joint_front_left" type="continuous">
+        <!-- <dynamics damping="0.0" friction="0.0"/> -->
+        <axis xyz="0 0 1"/>
+    </joint>
+    <joint name="wheel_joint_front_left" type="fixed">
         <parent link="left_bar"/>
         <child link="wheel_link_front_left"/>
         <origin xyz="-0.0254 0.10795 0" rpy="${-90*d2r} 0 ${90*d2r}"/>
-        <dynamics damping="0.0" friction="0.0"/>
-        <axis xyz="0 0 1"/>
-    </joint>
-    <joint name="wheel_joint_front_right" type="continuous">
+        <!-- <dynamics damping="0.0" friction="0.0"/> -->
+        <axis xyz="0 0 1"/>
+    </joint>
+    <joint name="wheel_joint_front_right" type="fixed">
         <parent link="right_bar"/>
         <child link="wheel_link_front_right"/>
         <origin xyz="0.0254 0.10795 0" rpy="${-90*d2r} 0 ${90*d2r}"/>
-        <dynamics damping="0.0" friction="0.0"/>
-        <axis xyz="0 0 1"/>
-    </joint>
-        <joint name="wheel_joint_middle_left" type="continuous">
+        <!-- <dynamics damping="0.0" friction="0.0"/> -->
+        <axis xyz="0 0 1"/>
+    </joint>
+        <joint name="wheel_joint_middle_left" type="fixed">
         <parent link="left_bar"/>
         <child link="wheel_link_middle_left"/>
         <origin xyz="-0.0254 0 0" rpy="${-90*d2r} 0 ${90*d2r}"/>
-        <dynamics damping="0.0" friction="0.0"/>
-        <axis xyz="0 0 1"/>
-    </joint>
-    <joint name="wheel_joint_middle_right" type="continuous">
+        <!-- <dynamics damping="0.0" friction="0.0"/> -->
+        <axis xyz="0 0 1"/>
+    </joint>
+    <joint name="wheel_joint_middle_right" type="fixed">
         <parent link="right_bar"/>
         <child link="wheel_link_middle_right"/>
         <origin xyz="0.0254 0 0" rpy="${-90*d2r} 0 ${90*d2r}"/>
-        <dynamics damping="0.0" friction="0.0"/>
-        <axis xyz="0 0 1"/>
-    </joint>
+        <!-- <dynamics damping="0.0" friction="0.0"/> -->
+        <axis xyz="0 0 1"/>
+    </joint>
+<gazebo reference= "base_link">
+      <collision>
+      <geometry>
+        <box size= "0 0 0" />
+      </geometry>
+          <surface>
+        <friction>
+          <ode>
+        <mu>0.5</mu>
+        <mu2>0.01</mu2>
+        <fdir1>1 0 0</fdir1>
+          </ode>
+        </friction>
+      </surface>
+    </collision>
+  </gazebo>
+  <!-- <gazebo reference= "back_bar">
+      <collision>
+      <geometry>
+        <box size= "0.0127 0.3302 0.0254" />
+      </geometry>
+          <surface>
+        <friction>
+          <ode>
+        <mu>0.01</mu>
+        <mu2>1.0</mu2>
+        <fdir1>1 0 0</fdir1>
+          </ode>
+        </friction>
+      </surface>
+    </collision>
+  </gazebo>
+  <gazebo reference= "left_bar">
+      <collision>
+      <geometry>
+        <box size= "0.0127 0.3302 0.0254" />
+      </geometry>
+          <surface>
+        <friction>
+          <ode>
+        <mu>0.01</mu>
+        <mu2>1.0</mu2>
+        <fdir1>1 0 0</fdir1>
+          </ode>
+        </friction>
+      </surface>
+    </collision>
+  </gazebo>
+    <gazebo reference= "right_bar">
+      <collision>
+      <geometry>
+        <box size= "0.0127 0.3302 0.0254" />
+      </geometry>
+          <surface>
+        <friction>
+          <ode>
+        <mu>0.01</mu>
+        <mu2>1.0</mu2>
+        <fdir1>1 0 0</fdir1>
+          </ode>
+        </friction>
+      </surface>
+    </collision>
+  </gazebo> -->
 </robot>
