Commit message: changes to comments

File: 04_Sim/ghost_sim_examples/urdf/tank_macros.xacro (robot description, xacro)
@@ -2,5 +2,5 @@
 <robot xmlns:xacro="http://www.ros.org/wiki/xacro">
     <!-- Wheel Macro -->
-    <xacro:macro name="wheel_macro" params="id r_wheel width_wheel collision_factor">
+    <xacro:macro name="wheel_macro" params="id r_wheel width_wheel collision_factor mu mu2 izz">
     <link name="wheel_link_${id}">
             <visual>
@@ -17,12 +17,4 @@
                     <cylinder radius="${r_wheel}" length="${width_wheel/collision_factor}"/>
                 </geometry>
-          <surface>
-        <friction>
-          <ode>
-         <mu>0.01</mu>
-            <mu2>1.0</mu2>
-          </ode>
-        </friction>
-      </surface>
             </collision>
             <!--Inertia estimated for solid cylinder of radius 2.5" and height 1" with mass 1 lb-->
@@ -33,27 +25,7 @@
                     ixx="0.000482" ixy="0.0" ixz="0.0"
                     iyy="0.000482" iyz="0.0"
-                    izz="0.000914"/>
+                    izz="${izz}"/>
             </inertial>
     </link>
-    <gazebo reference="wheel_${id}">
-        <collision>
-            <origin xyz="0 0 0" rpy="0 0 0"/>
-            <geometry>
-                <cylinder>
-                    <radius>${r_wheel}</radius>
-                    <length>${width_wheel/collision_factor}</length>
-                </cylinder>
-            </geometry>
-            <surface>
-                <friction>
-                    <torsional>
-                        <coefficient>1.0</coefficient>
-                        <patch_radius>0.01</patch_radius>
-                    </torsional>
-                </friction>
-            </surface>
-        </collision>
-        <material>Gazebo/White</material>
-    </gazebo>
     <gazebo reference="wheel_link_${id}">
         <collision>
@@ -67,13 +39,9 @@
             <surface>
                 <friction>
-          <ode>
-        <mu>0.5</mu>
-        <mu2>0.01</mu2>
-        <fdir1>1 0 0</fdir1>
-          </ode>
-                    <!-- <torsional>
-                        <coefficient>1.0</coefficient>
-                        <patch_radius>0.01</patch_radius>
-                    </torsional> -->
+                <ode>
+                    <mu>"${mu}"</mu>
+                    <mu2>"${mu2}"</mu2>
+                    <fdir1>1 0 0</fdir1>
+                </ode>
                 </friction>
             </surface>

File: 04_Sim/ghost_sim_examples/urdf/tankbot.xacro (robot description, xacro)
@@ -8,4 +8,7 @@
     <xacro:property name="com_radius" value="0.02"/>
     <xacro:property name="d2r" value="${3.14159/180}"/>
+    <xacro:property name="mu" value="0.01"/>
+    <xacro:property name="mu2" value="1.0"/>
+    <xacro:property name="izz" value="0.000914"/>
      <material name="white">
         <color rgba="1 1 1 1"/>
@@ -25,12 +28,4 @@
             <box size="0 0 0"/>
         </geometry>
-          <surface>
-        <friction>
-          <ode>
-         <mu>0.01</mu>
-            <mu2>1.0</mu2>
-          </ode>
-        </friction>
-      </surface>
         </collision>
         <inertial>
@@ -131,11 +126,11 @@
     </joint>
  <!--Wheel Modules-->
-    <xacro:wheel_macro id="front_left" r_wheel="${r_wheel}" width_wheel="${width_wheel}"   collision_factor="8"></xacro:wheel_macro>
-    <xacro:wheel_macro id="front_right" r_wheel="${r_wheel}" width_wheel="${width_wheel}"  collision_factor="8"></xacro:wheel_macro>
-    <xacro:wheel_macro id="back_left" r_wheel="${r_wheel}" width_wheel="${width_wheel}"  collision_factor="8"></xacro:wheel_macro>
-    <xacro:wheel_macro id="back_right" r_wheel="${r_wheel}" width_wheel="${width_wheel}"   collision_factor="8"></xacro:wheel_macro>
-    <xacro:wheel_macro id="middle_left" r_wheel="${r_wheel}" width_wheel="${width_wheel}"   collision_factor="8"></xacro:wheel_macro>
-    <xacro:wheel_macro id="middle_right" r_wheel="${r_wheel}" width_wheel="${width_wheel}"   collision_factor="8"></xacro:wheel_macro>
-    <joint name="wheel_joint_back_left" type="fixed">
+    <xacro:wheel_macro id="front_left" r_wheel="${r_wheel}" width_wheel="${width_wheel}"   collision_factor="8" mu="${mu}" mu2="${mu2}" izz="${izz}"></xacro:wheel_macro>
+    <xacro:wheel_macro id="front_right" r_wheel="${r_wheel}" width_wheel="${width_wheel}"  collision_factor="8" mu="${mu}" mu2="${mu2}" izz="${izz}"></xacro:wheel_macro>
+    <xacro:wheel_macro id="back_left" r_wheel="${r_wheel}" width_wheel="${width_wheel}"  collision_factor="8" mu="${mu}" mu2="${mu2}" izz="${izz}"></xacro:wheel_macro>
+    <xacro:wheel_macro id="back_right" r_wheel="${r_wheel}" width_wheel="${width_wheel}"   collision_factor="8" mu="${mu}" mu2="${mu2}" izz="${izz}"></xacro:wheel_macro>
+    <xacro:wheel_macro id="middle_left" r_wheel="${r_wheel}" width_wheel="${width_wheel}"   collision_factor="8" mu="${mu}" mu2="${mu2}" izz="${izz}"></xacro:wheel_macro>
+    <xacro:wheel_macro id="middle_right" r_wheel="${r_wheel}" width_wheel="${width_wheel}"   collision_factor="8" mu="${mu}" mu2="${mu2}" izz="${izz}"></xacro:wheel_macro>
+    <joint name="wheel_joint_back_left" type="continuous">
         <parent link="left_bar"/>
         <child link="wheel_link_back_left"/>
@@ -144,5 +139,5 @@
         <axis xyz="0 0 1"/>
     </joint>
-    <joint name="wheel_joint_back_right" type="fixed">
+    <joint name="wheel_joint_back_right" type="continuous">
         <parent link="right_bar"/>
         <child link="wheel_link_back_right"/>
@@ -151,5 +146,5 @@
         <axis xyz="0 0 1"/>
     </joint>
-    <joint name="wheel_joint_front_left" type="fixed">
+    <joint name="wheel_joint_front_left" type="continuous">
         <parent link="left_bar"/>
         <child link="wheel_link_front_left"/>
@@ -158,5 +153,5 @@
         <axis xyz="0 0 1"/>
     </joint>
-    <joint name="wheel_joint_front_right" type="fixed">
+    <joint name="wheel_joint_front_right" type="continuous">
         <parent link="right_bar"/>
         <child link="wheel_link_front_right"/>
@@ -165,5 +160,5 @@
         <axis xyz="0 0 1"/>
     </joint>
-        <joint name="wheel_joint_middle_left" type="fixed">
+        <joint name="wheel_joint_middle_left" type="continuous">
         <parent link="left_bar"/>
         <child link="wheel_link_middle_left"/>
@@ -172,5 +167,5 @@
         <axis xyz="0 0 1"/>
     </joint>
-    <joint name="wheel_joint_middle_right" type="fixed">
+    <joint name="wheel_joint_middle_right" type="continuous">
         <parent link="right_bar"/>
         <child link="wheel_link_middle_right"/>
@@ -179,67 +174,3 @@
         <axis xyz="0 0 1"/>
     </joint>
-<gazebo reference= "base_link">
-      <collision>
-      <geometry>
-        <box size= "0 0 0" />
-      </geometry>
-          <surface>
-        <friction>
-          <ode>
-        <mu>0.5</mu>
-        <mu2>0.01</mu2>
-        <fdir1>1 0 0</fdir1>
-          </ode>
-        </friction>
-      </surface>
-    </collision>
-  </gazebo>
-  <!-- <gazebo reference= "back_bar">
-      <collision>
-      <geometry>
-        <box size= "0.0127 0.3302 0.0254" />
-      </geometry>
-          <surface>
-        <friction>
-          <ode>
-        <mu>0.01</mu>
-        <mu2>1.0</mu2>
-        <fdir1>1 0 0</fdir1>
-          </ode>
-        </friction>
-      </surface>
-    </collision>
-  </gazebo>
-  <gazebo reference= "left_bar">
-      <collision>
-      <geometry>
-        <box size= "0.0127 0.3302 0.0254" />
-      </geometry>
-          <surface>
-        <friction>
-          <ode>
-        <mu>0.01</mu>
-        <mu2>1.0</mu2>
-        <fdir1>1 0 0</fdir1>
-          </ode>
-        </friction>
-      </surface>
-    </collision>
-  </gazebo>
-    <gazebo reference= "right_bar">
-      <collision>
-      <geometry>
-        <box size= "0.0127 0.3302 0.0254" />
-      </geometry>
-          <surface>
-        <friction>
-          <ode>
-        <mu>0.01</mu>
-        <mu2>1.0</mu2>
-        <fdir1>1 0 0</fdir1>
-          </ode>
-        </friction>
-      </surface>
-    </collision>
-  </gazebo> -->
 </robot>

Commit message: plugin as of now

File: 04_Sim/ghost_sim_examples/urdf/tank_macros.xacro (robot description, xacro)
@@ -2,5 +2,5 @@
 <robot xmlns:xacro="http://www.ros.org/wiki/xacro">
     <!-- Wheel Macro -->
-    <xacro:macro name="wheel_macro" params="id r_wheel width_wheel collision_factor mu mu2 izz">
+    <xacro:macro name="wheel_macro" params="id r_wheel width_wheel collision_factor izz">
     <link name="wheel_link_${id}">
             <visual>
@@ -21,8 +21,8 @@
             <inertial>
                 <origin xyz="0 0 0" rpy="0 0 0"/>
-                <mass value="0.4545"/>
+                <mass value="22.6796"/> <!--4.53592, ixx=0.004819, iyy=0.004819, izz= 0.009147-->
                 <inertia
-                    ixx="0.000482" ixy="0.0" ixz="0.0"
-                    iyy="0.000482" iyz="0.0"
+                    ixx="0.0481935" ixy="0.0" ixz="0.0"
+                    iyy="0.0481935" iyz="0.0"
                     izz="${izz}"/>
             </inertial>
@@ -40,6 +40,6 @@
                 <friction>
                 <ode>
-                    <mu>"${mu}"</mu>
-                    <mu2>"${mu2}"</mu2>
+                    <mu>1.0</mu> <!--1.0-->
+                    <mu2>0.1</mu2> <!--0.1-->
                     <fdir1>1 0 0</fdir1>
                 </ode>

File: 04_Sim/ghost_sim_examples/urdf/tankbot.xacro (robot description, xacro)
@@ -8,7 +8,7 @@
     <xacro:property name="com_radius" value="0.02"/>
     <xacro:property name="d2r" value="${3.14159/180}"/>
-    <xacro:property name="mu" value="0.01"/>
-    <xacro:property name="mu2" value="1.0"/>
-    <xacro:property name="izz" value="0.000914"/>
+    <!-- <xacro:property name="mu" value="0.01"/>
+    <xacro:property name="mu2" value="1.0"/> -->
+    <xacro:property name="izz" value="0.0457126"/>
      <material name="white">
         <color rgba="1 1 1 1"/>
@@ -126,15 +126,15 @@
     </joint>
  <!--Wheel Modules-->
-    <xacro:wheel_macro id="front_left" r_wheel="${r_wheel}" width_wheel="${width_wheel}"   collision_factor="8" mu="${mu}" mu2="${mu2}" izz="${izz}"></xacro:wheel_macro>
-    <xacro:wheel_macro id="front_right" r_wheel="${r_wheel}" width_wheel="${width_wheel}"  collision_factor="8" mu="${mu}" mu2="${mu2}" izz="${izz}"></xacro:wheel_macro>
-    <xacro:wheel_macro id="back_left" r_wheel="${r_wheel}" width_wheel="${width_wheel}"  collision_factor="8" mu="${mu}" mu2="${mu2}" izz="${izz}"></xacro:wheel_macro>
-    <xacro:wheel_macro id="back_right" r_wheel="${r_wheel}" width_wheel="${width_wheel}"   collision_factor="8" mu="${mu}" mu2="${mu2}" izz="${izz}"></xacro:wheel_macro>
-    <xacro:wheel_macro id="middle_left" r_wheel="${r_wheel}" width_wheel="${width_wheel}"   collision_factor="8" mu="${mu}" mu2="${mu2}" izz="${izz}"></xacro:wheel_macro>
-    <xacro:wheel_macro id="middle_right" r_wheel="${r_wheel}" width_wheel="${width_wheel}"   collision_factor="8" mu="${mu}" mu2="${mu2}" izz="${izz}"></xacro:wheel_macro>
+    <xacro:wheel_macro id="front_left" r_wheel="${r_wheel}" width_wheel="${width_wheel}"   collision_factor="8"  izz="${izz}"></xacro:wheel_macro>
+    <xacro:wheel_macro id="front_right" r_wheel="${r_wheel}" width_wheel="${width_wheel}"  collision_factor="8"  izz="${izz}"></xacro:wheel_macro>
+    <xacro:wheel_macro id="back_left" r_wheel="${r_wheel}" width_wheel="${width_wheel}"  collision_factor="8"  izz="${izz}"></xacro:wheel_macro>
+    <xacro:wheel_macro id="back_right" r_wheel="${r_wheel}" width_wheel="${width_wheel}"   collision_factor="8"  izz="${izz}"></xacro:wheel_macro>
+    <xacro:wheel_macro id="middle_left" r_wheel="${r_wheel}" width_wheel="${width_wheel}"   collision_factor="8"  izz="${izz}"></xacro:wheel_macro>
+    <xacro:wheel_macro id="middle_right" r_wheel="${r_wheel}" width_wheel="${width_wheel}"   collision_factor="8"  izz="${izz}"></xacro:wheel_macro>
     <joint name="wheel_joint_back_left" type="continuous">
         <parent link="left_bar"/>
         <child link="wheel_link_back_left"/>
         <origin xyz="-0.0254 -0.10795 0" rpy="${-90*d2r} 0 ${90*d2r}"/>
-        <!-- <dynamics damping="0.0" friction="0.0"/> -->
+        <!-- <dynamics damping="0.2" friction="0.2"/> -->
         <axis xyz="0 0 1"/>
     </joint>
@@ -143,5 +143,5 @@
         <child link="wheel_link_back_right"/>
         <origin xyz="0.0254 -0.10795 0" rpy="${-90*d2r} 0 ${90*d2r}"/>
-        <!-- <dynamics damping="0.0" friction="0.0"/> -->
+        <!-- <dynamics damping="0.2" friction="0.2"/> -->
         <axis xyz="0 0 1"/>
     </joint>
@@ -150,5 +150,5 @@
         <child link="wheel_link_front_left"/>
         <origin xyz="-0.0254 0.10795 0" rpy="${-90*d2r} 0 ${90*d2r}"/>
-        <!-- <dynamics damping="0.0" friction="0.0"/> -->
+        <!-- <dynamics damping="0.2" friction="0.2"/> -->
         <axis xyz="0 0 1"/>
     </joint>
@@ -157,5 +157,5 @@
         <child link="wheel_link_front_right"/>
         <origin xyz="0.0254 0.10795 0" rpy="${-90*d2r} 0 ${90*d2r}"/>
-        <!-- <dynamics damping="0.0" friction="0.0"/> -->
+        <!-- <dynamics damping="0.1" friction="0.1"/> -->
         <axis xyz="0 0 1"/>
     </joint>
@@ -164,5 +164,5 @@
         <child link="wheel_link_middle_left"/>
         <origin xyz="-0.0254 0 0" rpy="${-90*d2r} 0 ${90*d2r}"/>
-        <!-- <dynamics damping="0.0" friction="0.0"/> -->
+        <!-- <dynamics damping="0.1" friction="0.1"/> -->
         <axis xyz="0 0 1"/>
     </joint>
@@ -171,6 +171,31 @@
         <child link="wheel_link_middle_right"/>
         <origin xyz="0.0254 0 0" rpy="${-90*d2r} 0 ${90*d2r}"/>
-        <!-- <dynamics damping="0.0" friction="0.0"/> -->
-        <axis xyz="0 0 1"/>
-    </joint>
+        <!-- <dynamics damping="0.1" friction="0.1"/>  -->
+        <axis xyz="0 0 1"/>
+    </joint>
+<gazebo>
+<plugin name="gazebo_torque_plugin" filename="libgazebo_torque_plugin.so">
+            <free_speed>130</free_speed>
+            <stall_torque>4.5</stall_torque>
+            <free_current>0.1</free_current>
+            <stall_current>4.5</stall_current>
+            <nominal_voltage>12.0</nominal_voltage>
+            <gear_ratio>1.0</gear_ratio>
+            <joint_names>
+            wheel_joint_middle_left
+            wheel_joint_middle_right
+            </joint_names>
+            <!-- Motor names must be formatted in this manner in order to index actuator jacobian -->
+            <motor_names>
+                DRIVE_LEFT_FRONT_LEFT_MOTOR
+                DRIVE_RIGHT_FRONT_LEFT_MOTOR
+                DRIVE_LEFT_BACK_LEFT_MOTOR
+                DRIVE_RIGHT_BACK_LEFT_MOTOR
+            </motor_names>
+            <actuator_jacobian>
+                0.5     0.5      0           0
+                0        0      0.5         0.5
+            </actuator_jacobian>
+</plugin>
+</gazebo>
 </robot>
